File: pcb/pcb.kicad_sch (KiCad schematic)
At the start: 13 parts, among them J1 Conn_Coaxial, U1 XIAO-nRF52840-SMD, U2 NEO-M9V-20B, U3 AP2112K-3.3

Commit message: first version pcb done
Connections:
- net GND: now also U1.2 (P0.03_A1_D1)
- net uart_tx: now reaches R1.1, U2.20 (TXD/SPI_MISO)
- net uart_tx: now also U1.7 (P1.11_D6_TX); no longer U1.8 (P1.12_D7_RX)
- net at C2.1, C3.2, C4.1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: no longer L1.1
- net uart_rx: now reaches R2.1, U2.21 (RXD/SPI_MOSI)
- net uart_rx: now also U1.8 (P1.12_D7_RX); no longer U1.7 (P1.11_D6_TX)
- net at U2.9 (VCC_RF): now also L1.1
- no-connect marks 1 -> 34
Other:
- moved on the sheet: L1, U1
