File: pcb/pcb.kicad_sch (KiCad schematic)
At the start: 20 parts, among them J1 Conn_Coaxial, U1 XIAO-nRF52840-SMD, U2 NEO-M9V-20B, U3 AP2112K-3.3, U4 MCP73831-2-OT

Commit message: Update pcb from remove safeboot pull up
Connections:
- net at R5.1, U2.8 (~{RESET}): no longer U2.1 (~{SAFEBOOT})
- no-connect marks 26 -> 27
Changed lines of the file:
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@@
-	)
-	(junction
-		(at 148.59 85.09)
-		(diameter 0)
-		(color 0 0 0 0)
 	)
 	(junction
@@
 	)
 	(no_connect
+		(at 148.59 90.17)
+	)
+	(no_connect
 		(at 148.59 115.57)
 	)
@@
 		)
 		(stroke
-			(width 0)
-			(type default)
-		)
-	)
-	(wire
-		(pts
-			(xy 148.59 85.09) (xy 148.59 90.17)
-		)
-		(stroke
