File: pcb/v2_pcb/stm32power.kicad_sch (KiCad schematic)
At the start: 14 parts, among them U1 STM32N645I0H3Q

Commit message: start pcb v2
Parts:
- removed C1, C2: 100nF, symbol Device:C_Small
- removed C10, C11, C12, C3, C4, C7, C8, C9: 1uF, symbol Device:C_Small
- removed C5, C6: 10uF, symbol Device:C_Small
- removed L1: 2.2nH, symbol Device:L
- removed U1: STM32N645I0H3Q, VFBGA178_12X12_STM, symbol stm32n645i0:STM32N645I0H3Q
- added C169, C28, C36, C39, C40, C46, C47, C48, C50, C52, C54, C55, C58, C59, C64, C66, C67, C71, C72, C73, C74, C75, C76, C77, C78, C79, C80: 100nF, symbol Device:C_Small
- added C170, C176, C177, C178, C179: 22uF, symbol Device:C_Small
- added C29, C35: 10uF, symbol Device:C_Small
- added C34: 4.7uF, symbol Device:C_Small
- added C37: 2.2nF, symbol Device:C_Small
- added C38, C41, C43, C44, C45, C51, C57, C60, C61, C63, C65, C68, C69, C70: 1uF, symbol Device:C_Small
- added L4: 2.2nH, symbol Device:L_Small
- added L7: 1.0uH, symbol Device:L_Small
- added L8: 18R @ 100MHz, symbol Device:L_Small
- added R148, R159, R167, R173, R22, R27: 0R, symbol Device:R_Small_US
- added R168: 50mH, symbol Device:R_Small_US
- added R220: 2R, symbol Device:R_Small_US
- added U2: STM32N657X0H3Q, VFBGA264_14X14_STM, symbol noob:STM32N657X0H3Q
Connections:
- net GND: now also C169.1, C176.1, C177.2, C178.1, C179.1, C28.2, C29.2, C34.2, C35.2, C36.1, C37.2, C38.1, C39.1, C40.1, C41.2, C43.1, C44.1, C45.2, C46.1, C47.1, C48.2, C50.1, C51.1, C52.2, C54.1, C55.1, C57.1, C58.1, C59.1, C60.1, C61.1, C63.1, C64.1, C65.1, C66.1, C67.1, C68.1, C69.1, C70.1, C71.1, C72.1, C73.1, C74.1, C75.1, C76.1, C77.1, C78.1, C79.1, C80.1, U2.A17 (VSS), U2.F10 (VSS), U2.F11 (VSS), U2.F12 (VSS), U2.F2 (VSSAPMU), U2.F7 (VSS), U2.G12 (VSS), U2.G6 (VSSAON), U2.H1 (VSSSMPS), U2.H2 (VSSSMPS), U2.H3 (VSSSMPS), U2.H4 (VSSSMPS), U2.H5 (VSSSMPS), U2.H6 (VSSSMPS), U2.K12 (VSS), U2.M10 (VSS), U2.M12 (VSS), U2.M13 (VSS), U2.M6 (VSSA), U2.M8 (VSS), U2.N11 (VSS), U2.N5 (VSS), U2.N7 (VSS), U2.N9 (VSS), U2.T2 (VREF-), U2.U1 (VSS), U2.U17 (VSS)
- new net: L7.1, R220.1, U2.J1 (VLXSMPS), U2.J2 (VLXSMPS), U2.J3 (VLXSMPS), U2.J4 (VLXSMPS), U2.J5 (VLXSMPS), U2.J6 (VLXSMPS)
- new net: C37.1, R220.2
- new net: C29.1, C35.1, C41.1, C45.1, C48.1, C52.1, L4.2, U2.K1 (VDDSMPS), U2.K2 (VDDSMPS), U2.K3 (VDDSMPS), U2.K4 (VDDSMPS), U2.K5 (VDDSMPS), U2.K6 (VDDSMPS)
- new net: C46.2, C47.2, C50.2, C54.2, C71.2, C74.2, C77.2, C78.2, C79.2, C80.2
- new net: C55.2, C58.2, C66.2, C67.2, C72.2, C73.2, C75.2, C76.2
- new net: C38.2, C39.2
- new net: C44.2, C51.2, C57.2, C60.2, C61.2, C63.2, C65.2, C68.2, C69.2, C70.2
- new net: C34.1, U2.F1 (V08CAP)
- new net: C43.2, R159.2, U2.A4 (VDD33USB)
- new net: C59.2, C64.2
- new net: C28.1, U2.E1 (VBAT)
- new net: U2.C5 (VDDA18USB), U2.M5 (VDDA18PLL), U2.N6 (VDDA18ADC), U2.R5 (VDDA18CSI)
- new net: U2.E8 (VDDIO4), U2.F8 (VDDIO4)
- new net: U2.E9 (VDDIO5), U2.F9 (VDDIO5)
- new net: R148.2, U2.F6 (VDDA18AON)
- new net: C169.2, U2.G1 (VDDA18PMU)
- new net: U2.G13 (VDD), U2.H12 (VDD), U2.H13 (VDD), U2.J12 (VDD), U2.J13 (VDD), U2.K13 (VDD)
- new net: U2.L12 (VDDCORE), U2.L6 (VDDCORE), U2.M11 (VDDCORE), U2.M7 (VDDCORE), U2.M9 (VDDCORE), U2.N10 (VDDCORE), U2.N12 (VDDCORE), U2.N8 (VDDCORE), U2.P11 (VDDCORE), U2.R4 (VDDCSI)
- new net: U2.L13 (VDDIO2), U2.L14 (VDDIO2), U2.M14 (VDDIO2), U2.M15 (VDDIO2), U2.N13 (VDDIO3), U2.P13 (VDDIO3)
- new net MCUPower: C170.1, C170.2, C176.2, C177.1, C178.2, C179.2, L7.2, R167.1, R167.2, R168.1, R168.2, R22.2, U2.G2 (VFBSMPS)

Commit message: add ram
Connections:
- net MCUPower: no longer C170.1, C170.2, C176.2, C177.1, C178.2, C179.2, L7.2, R167.1, R167.2, R168.1, R168.2, R22.2, U2.G2 (VFBSMPS)
- new net I_SENS_VDDCORE_N: C170.1, R167.1, R168.1, R22.2, U2.G2 (VFBSMPS)
- new net I_SENS_VDDCORE_P: C170.2, C176.2, C177.1, C178.2, C179.2, L7.2, R167.2, R168.2
Changed lines of the file:
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@@
-	)
-	(junction
-		(at 50.8 171.45)
-		(diameter 0)
-		(color 0 0 0 0)
 	)
 	(junction
@@
 		)
 	)
+	(bus
+		(pts
+			(xy 41.91 171.45) (xy 50.8 171.45)
+		)
+		(stroke
+			(width 0)
+			(type default)
+		)
+	)
 	(wire
 		(pts
@@
 	(wire
 		(pts
-			(xy 41.91 171.45) (xy 50.8 171.45)
-		)
-		(stroke
-			(width 0)
-			(type default)
-		)
-	)
-	(wire
-		(pts
 			(xy 140.97 133.35) (xy 143.51 133.35)
 		)
@@
 	(wire
 		(pts
+			(xy 50.8 171.45) (xy 69.85 171.45)
+		)
+		(stroke
+			(width 0)
+			(type default)
+		)
+	)
+	(wire
+		(pts
 			(xy 82.55 41.91) (xy 85.09 41.91)
 		)
@@
 		)
 	)
+	(bus
+		(pts
+			(xy 50.8 168.91) (xy 50.8 171.45)
+		)
+		(stroke
+			(width 0)
+			(type default)
+		)
+	)
 	(wire
 		(pts
@@
 	(wire
 		(pts
-			(xy 50.8 168.91) (xy 50.8 171.45)
-		)
-		(stroke
-			(width 0)
-			(type default)
-		)
-	)
-	(wire
-		(pts
 			(xy 140.97 146.05) (xy 143.51 146.05)
 		)
@@
 	(wire
 		(pts
-			(xy 50.8 171.45) (xy 69.85 171.45)
-		)
-		(stroke
-			(width 0)
-			(type default)
-		)
-	)
-	(wire
-		(pts
 			(xy 82.55 82.55) (xy 85.09 82.55)
 		)
@@
 	)
 	(label "I_SENS_VDDCORE_P"
-		(at 234.95 34.29 0)
+		(at 252.73 34.29 180)
 		(effects
 			(font
 				(size 1.27 1.27)
 			)
-			(justify left bottom)
+			(justify right bottom)
 		)
 	)
 	(label "I_SENS_VDDCORE_N"
-		(at 154.94 57.15 0)
+		(at 172.72 57.15 180)
 		(effects
 			(font
 				(size 1.27 1.27)
 			)
-			(justify left bottom)
+			(justify right bottom)
 		)
 	)
 	(label "I_SENS_VDDCORE_P"
-		(at 52.07 168.91 0)
+		(at 69.85 168.91 180)
 		(effects
 			(font
 				(size 1.27 1.27)
 			)
-			(justify left bottom)
+			(justify right bottom)
 		)
 	)
 	(label "I_SENS_VDDCORE_N"
-		(at 52.07 171.45 0)
+		(at 69.85 171.45 180)
 		(effects
 			(font
 				(size 1.27 1.27)
 			)
-			(justify left bottom)
+			(justify right bottom)
 		)
 	)
 	(label "I_SENS_VDDCORE_P"
-		(at 167.64 44.45 0)
+		(at 186.69 44.45 180)
 		(effects
 			(font
 				(size 1.27 1.27)
 			)
-			(justify left bottom)
-		)
-	)
+			(justify right bottom)
+		)
+	)
