File: pcb/v2_pcb/stm32power.kicad_sch (KiCad schematic)
At the start: 62 parts, among them U2 STM32N657X0H3Q

Commit message: add rpls for 1v8, 5v
Parts:
- R168: value 50mH -> 50mR (DNP); now not fitted
Changed lines of the file:
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@@
 			)
 		)
-		(property "Value" "VDDIO"
+		(property "Value" "+3V3_MAIN"
 			(at 78.74 25.4 90)
 			(show_name no)
@@
 			)
 		)
-		(property "Value" "VDDA1V8_AON"
+		(property "Value" "+1V8_AON"
 			(at 237.49 78.74 0)
 			(show_name no)
@@
 			)
 		)
-		(property "Value" "VDD3V3"
+		(property "Value" "+3V3_MAIN"
 			(at 49.53 123.1899 90)
 			(show_name no)
@@
 			)
 		)
-		(property "Value" "VDD1V8"
+		(property "Value" "+1V8_RUN"
 			(at 78.74 163.83 0)
 			(show_name no)
@@
 			)
 		)
-		(property "Value" "VDDA1V8"
+		(property "Value" "+1V8_RUN"
 			(at 76.2 46.9899 90)
 			(show_name no)
@@
 			)
 		)
-		(property "Value" "VREFP"
+		(property "Value" "+1V8_RUN"
 			(at 147.32 69.8499 90)
 			(show_name no)
@@
 			)
 		)
-		(property "Value" "VDDA1V8"
+		(property "Value" "+1V8_RUN"
 			(at 60.96 138.4299 90)
 			(show_name no)
@@
 			)
 		)
-		(property "Value" "VDDA1V8"
+		(property "Value" "+1V8_RUN"
 			(at 118.11 172.72 0)
 			(show_name no)
@@
 			)
 		)
-		(property "Value" "VDDIO"
+		(property "Value" "+3V3_MAIN"
 			(at 165.1 97.79 0)
 			(show_name no)
@@
 			)
 		)
-		(property "Value" "VDDIO"
+		(property "Value" "+3V3_MAIN"
 			(at 160.02 74.9299 90)
 			(show_name no)
@@
 			)
 		)
-		(property "Value" "VDDIO"
+		(property "Value" "+3V3_MAIN"
 			(at 76.2 62.2299 90)
 			(show_name no)
@@
 			)
 		)
-		(property "Value" "VDDA1V8"
+		(property "Value" "+1V8_RUN"
 			(at 78.74 181.61 0)
 			(show_name no)
@@
 			)
 		)
-		(property "Value" "VDDIO_SD"
+		(property "Value" "+3V3_MAIN"
 			(at 200.66 78.74 0)
 			(show_name no)
@@
 			)
 		)
-		(property "Value" "VDDIO_SD"
+		(property "Value" "+3V3_MAIN"
 			(at 76.2 67.3099 90)
 			(show_name no)
@@
 			)
 		)
-		(property "Value" "VDDA1V8"
+		(property "Value" "+1V8_RUN"
 			(at 165.1 115.57 0)
 			(show_name no)
@@
 			)
 		)
-		(property "Value" "VDD1V8"
+		(property "Value" "+1V8_RUN"
 			(at 20.32 110.4899 90)
 			(show_name no)
@@
 			)
 		)
-		(property "Value" "VREFP"
+		(property "Value" "+1V8_RUN"
 			(at 180.34 78.74 0)
 			(show_name no)
@@
 			)
 		)
-		(property "Value" "VREFP"
+		(property "Value" "+1V8_RUN"
 			(at 118.11 181.61 0)
 			(show_name no)
@@
 			)
 		)
-		(property "Value" "VDDA1V8_AON"
+		(property "Value" "+1V8_AON"
 			(at 39.37 128.27 0)
 			(show_name no)
@@
 		(on_board yes)
 		(in_pos_files yes)
-		(dnp no)
+		(dnp yes)
 		(fields_autoplaced yes)
 		(property "Reference" "R168"
@@
 			)
 		)
-		(property "Value" "50mH"
+		(property "Value" "50mR (DNP)"
 			(at 226.06 35.56 90)
 			(show_name no)

Commit message: pcb done
Parts:
- added C308: 1uF, Capacitor_SMD:C_0402_1005Metric, symbol Device:C_Small
- added C309: 100nF, Capacitor_SMD:C_0402_1005Metric, symbol Device:C_Small
- C169, C28, C36, C38, C39, C40, C41, C43, C44, C45, C46, C47, C48, C50, C51, C52, C54, C55, C57, C58, C59, C60, C61, C63, C64, C65, C66, C67, C68, C69, C70, C71, C72, C73, C74, C75, C76, C77, C78, C79, C80: footprint (none) -> Capacitor_SMD:C_0402_1005Metric
- C170, C176, C177, C178, C179, C29, C35: footprint (none) -> Capacitor_SMD:C_0805_2012Metric
- C34: footprint (none) -> Capacitor_SMD:C_0603_1608Metric
- C37: value 2.2nF -> 2.2nF 50V X7R; footprint (none) -> Capacitor_SMD:C_0402_1005Metric; Function (none) -> VLXSMPS series snubber capacitor; AN5967-rated 50V
- L4: footprint (none) -> Inductor_SMD:L_1210_3225Metric
- L7: value 1.0uH -> 1uH; footprint (none) -> Inductor_SMD:L_1008_2520Metric; Electrical Spec (none) -> 1uH +/-20%; DCR 42mR max; 30% L-drop current 4.3A; 40C-rise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; MPN (none) -> DFE252012P-1R0M=P2; Manufacturer (none) -> Murata
- L8: footprint (none) -> Inductor_SMD:L_0603_1608Metric_Pad1.05x0.95mm_HandSolder
- R148, R159, R220: footprint (none) -> Resistor_SMD:R_0402_1005Metric
- R167, R22: footprint (none) -> Resistor_SMD:R_1206_3216Metric
- R168: footprint (none) -> Resistor_SMD:R_2512_6332Metric; BOM Comments (none) -> Optional 50mR current-sense shunt; populate instead of R167; now fitted; now left out of the parts list
- R173: value 0R -> 0R DNP (alternate to L8); footprint (none) -> Resistor_SMD:R_0402_1005Metric; BOM Comments (none) -> Optional 0R bypass; populate instead of ferrite bead L8; now left out of the parts list
- R27: footprint (none) -> Resistor_SMD:R_0402_1005Metric; MPN (none) -> RC0402JR-070RL; Manufacturer (none) -> Yageo
- U1: renamed from U2; footprint VFBGA264_14X14_STM -> noob:VFBGA264_14X14_STM
Connections:
- net GND: now also C308.2, C309.2
- net +1V8_RUN: now reaches C46.2, C47.2, C50.2, C54.2, C71.2, C74.2, C77.2, C78.2, C79.2, C80.2
- net +1V8_RUN: now also C38.2, C39.2, L4.1, L8.1, R173.2, R27.1, U1.C5 (VDDA18USB), U1.L13 (VDDIO2), U1.L14 (VDDIO2), U1.M14 (VDDIO2), U1.M15 (VDDIO2), U1.M5 (VDDA18PLL), U1.N13 (VDDIO3), U1.N6 (VDDA18ADC), U1.P13 (VDDIO3), U1.R5 (VDDA18CSI)
- net VREFP: now reaches R27.2
- net VREFP: now also U1.U2 (VREF+), C308.1, C309.1
- net VDDCORE: now reaches R22.1
- net VDDCORE: now also C44.2, C51.2, C57.2, C60.2, C61.2, C63.2, C65.2, C68.2, C69.2, C70.2, U1.L12 (VDDCORE), U1.L6 (VDDCORE), U1.M11 (VDDCORE), U1.M7 (VDDCORE), U1.M9 (VDDCORE), U1.N10 (VDDCORE), U1.N12 (VDDCORE), U1.N8 (VDDCORE), U1.P11 (VDDCORE), U1.R4 (VDDCSI)
- net +3V3_MAIN: now reaches C55.2, C58.2, C66.2, C67.2, C72.2, C73.2, C75.2, C76.2
- net +3V3_MAIN: now also C28.1, C59.2, C64.2, R159.1, U1.E1 (VBAT), U1.E8 (VDDIO4), U1.E9 (VDDIO5), U1.F8 (VDDIO4), U1.F9 (VDDIO5), U1.G13 (VDD), U1.H12 (VDD), U1.H13 (VDD), U1.J12 (VDD), U1.J13 (VDD), U1.K13 (VDD)
- net +1V8_AON: now reaches C36.2
- net +1V8_AON: now also R148.1
- net VDDA18PMU: now reaches L8.2
- net VDDA18PMU: now also C169.2, R173.1, U1.G1 (VDDA18PMU)
- net VDDA18AON: now reaches R148.2, U1.F6 (VDDA18AON)
- net VDDA18AON: now also C40.2

Commit message: minor fixes
Parts:
- C169, C28, C309, C36, C39, C40, C46, C47, C48, C50, C52, C54, C55, C58, C59, C64, C66, C67, C71, C72, C73, C74, C75, C76, C77, C78, C79, C80: value 100nF -> 100nF 50V X7R; Dielectric (none) -> X7R; MPN (none) -> CGA2B3X7R1H104K050BE; Manufacturer (none) -> TDK; Qualification (none) -> AEC-Q200; Termination (none) -> Soft termination; Tolerance (none) -> ±10%; Voltage (none) -> 50 VDC
- C170, C176, C177, C178, C179: value 22uF -> 22uF 6.3V X7T; Dielectric (none) -> X7T; MPN (none) -> GCJ21BD70J226ME02L; Manufacturer (none) -> Murata; Qualification (none) -> AEC-Q200; Release_Status (none) -> Verify STM32 output bank effective capacitance; C170 is cro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; Termination (none) -> Soft termination; Tolerance (none) -> ±20%; Voltage (none) -> 6.3 VDC
- C29, C35: value 10uF -> 10uF 10V X7R; Dielectric (none) -> X7R; MPN (none) -> GCJ21BR71A106KE01L; Manufacturer (none) -> Murata; Qualification (none) -> AEC-Q200; Termination (none) -> Soft termination; Tolerance (none) -> ±10%; Voltage (none) -> 10 VDC
- C308, C38, C41, C43, C44, C45, C51, C57, C60, C61, C63, C65, C68, C69, C70: value 1uF -> 1uF 10V X7S; Dielectric (none) -> X7S; MPN (none) -> GCM155C71A105KE38D; Manufacturer (none) -> Murata; Qualification (none) -> AEC-Q200 powertrain/safety; Tolerance (none) -> ±10%; Voltage (none) -> 10 VDC
- C34: value 4.7uF -> 4.7uF 16V X7S; Dielectric (none) -> X7S; MPN (none) -> GCM188C71C475KE36D; Manufacturer (none) -> Murata; Qualification (none) -> AEC-Q200 powertrain/safety; Tolerance (none) -> ±10%; Voltage (none) -> 16 VDC
- C37: Dielectric (none) -> X7R; MPN (none) -> CGA2B2X7R1H222K050BE; Manufacturer (none) -> TDK; Qualification (none) -> AEC-Q200; Termination (none) -> Soft termination; Tolerance (none) -> ±10%; Voltage (none) -> 50 VDC
- L4: value 2.2nH -> 2.2nH 1A; footprint Inductor_SMD:L_1210_3225Metric -> open-race-v2:L_TDK_MHQ1005_1.0x0.6mm; DCR_Max (none) -> 60mR; Design_Note (none) -> STM32N6 VDDSMPS feed; use TDK recommended 0.35/0.50/0.65 mm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; MPN (none) -> MHQ1005P2N2BT000; Manufacturer (none) -> TDK; SRF_Min (none) -> 8GHz
- L8: value 18R @ 100MHz -> 22R @100MHz 8A; footprint Inductor_SMD:L_0603_1608Metric_Pad1.05x0.95mm_HandSolder -> Inductor_SMD:L_0603_1608Metric; DCR_Max (none) -> 4mR; Design_Note (none) -> STM32N6 supply ferrite; 8 A rating at 85 C, 5 A at 125 C; MPN (none) -> BLM18SN220TN1D; Manufacturer (none) -> Murata
- R148, R159: MPN (none) -> CRCW04020000Z0ED; Manufacturer (none) -> Vishay; Power (none) -> 1.5 A; ≤20 mΩ; TCR (none) -> N/A; Tolerance (none) -> Jumper
- R167, R22: MPN (none) -> WFZ120600000ZE66; Manufacturer (none) -> Vishay; Power (none) -> 38 A; ≤0.5 mΩ; TCR (none) -> N/A; Tolerance (none) -> Jumper
- R220: MPN (none) -> RCS04022R00FKED; Manufacturer (none) -> Vishay; Power (none) -> 0.20 W pulse-rated; TCR (none) -> ±100 ppm/K; Tolerance (none) -> ±1%
- R27: Power (none) -> 1 A rated / 2 A max; TCR (none) -> N/A; Tolerance (none) -> Jumper
