File: pcb/v2_pcb/HexaSPI_PSRAM.kicad_sch (KiCad schematic)
At the start: 0 parts

Commit message: add ram
Parts:
- added C141, C143: 4.7uF, symbol Device:C_Small
- added C142, C144: 100nF, symbol Device:C_Small
- added U3: APS512XXN-OB9-BG, APS512XXN-OB9-BG:BGA24C100P5X5_800X600X120, symbol noob:APS256XXN-OBR-BG
Connections:
- new net GND: C141.2, C142.2, C143.2, C144.2, U3.C1 (VSS)
- new net HEXASPI_CLK: U3.B2 (CLK)
- new net HEXASPI_DQS0: U3.C3 (DQS/DM0)
- new net HEXASPI_DQS1: U3.B3 (DQS/DM1)
- new net HEXASPI_IO0: U3.C2 (DQ8), U3.D3 (ADQ0)
- new net HEXASPI_IO1: U3.B1 (DQ9), U3.D2 (ADQ1)
- new net HEXASPI_IO2: U3.A2 (DQ10), U3.C4 (ADQ2)
- new net HEXASPI_IO3: U3.A4 (DQ11), U3.D4 (ADQ3)
- new net HEXASPI_IO4: U3.A5 (DQ12), U3.D5 (ADQ4)
- new net HEXASPI_IO5: U3.B4 (DQ13), U3.E3 (ADQ5)
- new net HEXASPI_IO6: U3.B5 (DQ14), U3.E2 (ADQ6)
- new net HEXASPI_NCS: U3.A3 (~{CE})
- new net VDD: C141.1, C142.1, C143.1, C144.1, U3.D1 (VDD), U3.E4 (VDD)
- new net VSS: U3.C5 (DQ15), U3.E1 (ADQ7), U3.E5 (VSS)
Other:
- note added: "100 nF/4.7µF decoupling for each pair C1/D1"
