File: pcb/v2_pcb/USB.kicad_sch (KiCad schematic)
At the start: 30 parts, among them IC1 AP33772SDKZ-13-FA01, J2 USB4105-GF-A, Q1 NMOS, Q2 NMOS, U24 TXS0104EPW, U25 TPS3808G01DBVR, U4 TPD8S300ARUKR

Commit message: minor fixes
Parts:
- added C255, C256: 1uF 25V X7R, Capacitor_SMD:C_0603_1608Metric, symbol Device:C_Small
- added D3: TVS2200DRVR, open-race-v2:WSON-6-1EP_2x2mm_P0.65mm_EP1x1.6mm_TVS2200, symbol Power_Protection:TVS2200DRV
- added U26: TLV75533PDBVR, Package_TO_SOT_SMD:SOT-23-5, symbol Regulator_Linear:TLV75533PDBV
- C2, C231, C232, C4: value 100nF -> 100nF 50V X7R; Dielectric (none) -> X7R; MPN (none) -> CGA3E2X7R1H104K080AE; Manufacturer (none) -> TDK; Qualification (none) -> AEC-Q200; Termination (none) -> Soft termination; Tolerance (none) -> ±10%; Voltage (none) -> 50 VDC
- C230: value 1uF 35V X7R -> 1uF 50V X7R; Dielectric (none) -> X7R; MPN (none) -> CGA4J3X7R1H105K125AE; Manufacturer (none) -> TDK; Qualification (none) -> AEC-Q200; Termination (none) -> Soft termination; Tolerance (none) -> ±10%; Voltage (none) -> 50 VDC
- C253: value 100nF 10V X7R -> 100nF 50V X7R; Dielectric (none) -> X7R; MPN (none) -> CGA3E2X7R1H104K080AE; Manufacturer (none) -> TDK; Qualification (none) -> AEC-Q200; Termination (none) -> Soft termination; Tolerance (none) -> ±10%; Voltage (none) -> 50 VDC
- C254: value 1nF 10V X7R -> 1nF 100V C0G; Dielectric (none) -> C0G; MPN (none) -> CGA3E2C0G2A102J080AE; Manufacturer (none) -> TDK; Qualification (none) -> AEC-Q200; Termination (none) -> Soft termination; Tolerance (none) -> ±5%; Voltage (none) -> 100 VDC
- C3, C6: value 1uF 10V X7R -> 1uF 50V X7R; Dielectric (none) -> X7R; MPN (none) -> CGA4J3X7R1H105K125AE; Manufacturer (none) -> TDK; Qualification (none) -> AEC-Q200; Termination (none) -> Soft termination; Tolerance (none) -> ±10%; Voltage (none) -> 50 VDC
- C5: Dielectric (none) -> X7R; MPN (none) -> CGA3E2X7R1H104K080AE; Manufacturer (none) -> TDK; Qualification (none) -> AEC-Q200; Termination (none) -> Soft termination; Tolerance (none) -> ±10%; Voltage (none) -> 50 VDC
- D1: value LTST-C190KGKT GREEN -> ASMT-RF45-AN002 YELLOW GREEN; Color (none) -> Yellow green; Current (none) -> 20 mA maximum; visual-qualify at fitted 1 kΩ drive; MPN LTST-C190KGKT -> ASMT-RF45-AN002; Manufacturer (none) -> Broadcom; Operating_Temperature (none) -> -40 to +100 °C; Qualification (none) -> Automotive qualified
- IC1: value AP33772SDKZ-13-FA01 -> AP33772SDKZ-13-FA02; footprint Package_DFN_QFN:WQFN-24-1EP_4x4mm_P0.5mm_EP2.45x2.45mm -> open-race-v2:WQFN-24-1EP_4x4mm_P0.5mm_EP2.70x2.70mm_AP33772S; symbol noob:AP33772SDKZ-13-FA01 -> noob:AP33772SDKZ-13-FA02; Design_Note (none) -> SPR/PPS-only build: pin 7 GPIO intentionally NC; pin 11 VSE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; MPN AP33772SDKZ-13-FA01 -> AP33772SDKZ-13-FA02; Manufacturer (none) -> Diodes Incorporated; Manufacturer_Part_Number AP33772SDKZ-13-FA01 -> AP33772SDKZ-13-FA02; Mouser Part Number 621-P33772SDKZ13FA01 -> (none); Mouser Price/Stock https://www.mouser.co.uk/ProductDetail/Diodes-Incorporated/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 -> (none)
- J2: Manufacturer (none) -> Global Connector Technology (GCT)
- Q1, Q2: value NMOS -> CSD18540Q5B
- R1: MPN (none) -> CRCW06036K20FKEA; Manufacturer (none) -> Vishay; Power (none) -> 0.10 W; TCR (none) -> ±100 ppm/K; Tolerance (none) -> ±1%
- R2: MPN (none) -> CRCW0603200RFKEA; Manufacturer (none) -> Vishay; Power (none) -> 0.10 W; TCR (none) -> ±100 ppm/K; Tolerance (none) -> ±1%
- R241, R242: MPN (none) -> CRCW06035K10FKEA; Manufacturer (none) -> Vishay; Power (none) -> 0.10 W; TCR (none) -> ±100 ppm/K; Tolerance (none) -> ±1%
- R243, R251, R5: MPN (none) -> CRCW060310K0FKEA; Manufacturer (none) -> Vishay; Power (none) -> 0.10 W; TCR (none) -> ±100 ppm/K; Tolerance (none) -> ±1%
- R249: MPN (none) -> CRCW0603100KFKEA; Manufacturer (none) -> Vishay; Power (none) -> 0.10 W; TCR (none) -> ±100 ppm/K; Tolerance (none) -> ±1%
- R250: MPN (none) -> CRCW060388K7FKEA; Manufacturer (none) -> Vishay; Power (none) -> 0.10 W; TCR (none) -> ±100 ppm/K; Tolerance (none) -> ±1%
- R3: Manufacturer (none) -> Vishay Dale; Power (none) -> 1.0 W at 70 °C; Qualification (none) -> AEC-Q200; TCR (none) -> ±75 ppm/K; Tolerance (none) -> ±1%
- R4: MPN (none) -> CRCW06031K00FKEA; Manufacturer (none) -> Vishay; Power (none) -> 0.10 W; TCR (none) -> ±100 ppm/K; Tolerance (none) -> ±1%
- TH1: Manufacturer (none) -> Murata
- U4: Manufacturer (none) -> Texas Instruments
Connections:
- net +3V3_MAIN: no longer C6.1, U4.10 (VPWR)
- net AP_ISENP: now also D3.4 (IN), D3.5 (IN), D3.6 (IN)
- net AP_V5V: now also C255.1, U26.1 (IN), U26.3 (EN)
- net AP_VCC: now also Q1.5 (D), Q1.6 (D), Q1.7 (D), Q1.8 (D); no longer Q1.1 (S), Q1.2 (S), Q1.3 (S)
- net GND: now also C255.2, C256.2, D3.1 (GND), D3.2 (GND), D3.3 (GND), D3.7 (GND), U26.2 (GND)
- net USB_PD_FET_COMMON: now also Q1.1 (S), Q1.2 (S), Q1.3 (S), Q2.1 (S), Q2.2 (S), Q2.3 (S); no longer Q1.5 (D), Q1.6 (D), Q1.7 (D), Q1.8 (D), Q2.5 (D), Q2.6 (D), Q2.7 (D), Q2.8 (D)
- net VBUS_PD: now also Q2.5 (D), Q2.6 (D), Q2.7 (D), Q2.8 (D); no longer Q2.1 (S), Q2.2 (S), Q2.3 (S)
- new net USB_PROT_3V3_AON: C256.1, C6.1, U26.5 (OUT), U4.10 (VPWR)
- no-connect marks 16 -> 17
Other:
- note added: "SPR ONLY: D3 TVS2200 prohibits 28 V EPR. Firmware must clear EPR_MODE_EN, accept only <=20 V PDOs, and validate VCC overshoot on the worst cable."
- note added: "USB PD RELEASE GATE — SPR/PPS ONLY: at startup write PDCONFIG=0x02 (clear EPR_MODE_EN); reject PDO8–13/AVS; never request >20.0 V. TPD8S300A is not EPR-rated."
- note removed: "USB PD POLICY: SPR/PPS only; firmware request <=20 V (21 V design ceiling). EPR MUST remain disabled."
