File: pcb/v2_pcb/STM32_MCU_IO.kicad_sch (KiCad schematic)
At the start: 24 parts, among them U1 STM32N657X0H3Q

Commit message: add rpls for 1v8, 5v
Changed lines of the file:
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@@
 			)
 		)
-		(property "Value" "VDDA1V8_AON"
+		(property "Value" "+1V8_AON"
 			(at 288.29 213.3599 90)
 			(show_name no)

Commit message: run load switch
Changed lines of the file:
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@@
 	)
 	(hierarchical_label "PWR_ON"
-		(shape input)
+		(shape output)
 		(at 284.48 208.28 0)
 		(effects

Commit message: pcb done
Parts:
- removed R32, R33, R34: 200R, symbol Device:R_Small_US
- added C300, C301, C302, C303: 8.2pF C0G (TUNE), Capacitor_SMD:C_0402_1005Metric, symbol Device:C_Small
- added C304: 100nF, Capacitor_SMD:C_0402_1005Metric, symbol Device:C_Small
- added R300, R301: 10k, Resistor_SMD:R_0402_1005Metric, symbol Device:R_Small_US
- added R304: 100k, Resistor_SMD:R_0402_1005Metric, symbol Device:R_Small_US
- added R320, R321, R322, R323, R324, R325: 22R, Resistor_SMD:R_0402_1005Metric, symbol Device:R_Small_US
- added R326: 200R 1%, Resistor_SMD:R_0402_1005Metric, symbol Device:R_Small_US
- added SW300: BOOT, Button_Switch_SMD:SW_Push_1P1T_NO_CK_KMR2, symbol Switch:SW_Push
- added Y1: NX2016SA-24MHZ-EXS00A-CS10820, Crystal:Crystal_SMD_2016-4Pin_2.0x1.6mm, symbol open-race-v2:Crystal_GND24_Separated
- added Y2: NX2012SA-32.768KHZ-EXS00A-MU00527, Crystal:Crystal_SMD_2012-2Pin_2.0x1.2mm, symbol Device:Crystal
- R44, R45, R46, R47, R48, R49, R50, R51, R53, R54, R55, R56, R57, R58, R59, R60, R61, R62, R63, R64: value Resistor -> 22R; footprint Library:R0402 -> Resistor_SMD:R_0402_1005Metric; ALTIUM_VALUE 0R -> (none); COMPONENTLINK1URL http://tunmcdsvn.tun.st.com/Component_Documentation_Library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 -> (none); COMPONENT_COUNTRY_OF_ORIGIN China -> (none); ID 2540 -> (none); INTERNAL_PART_NUMBER MCD-00052 -> (none); MANUFACTURER YAGEO -> (none); MANUFACTURER_PART_NUMBER RC0402JR-070RL -> (none); MPN (none) -> RC0402FR-0722RL; Manufacturer (none) -> Yageo; ORDER_CODE_DIGIKEY 311-0.0JRCT-ND -> (none); ORDER_CODE_FARNELL 9232516RL -> (none); ORDER_CODE_RS 9232516RL -> (none); PACKAGE 0402 -> (none); PART_PREFERENCE Recommended -> (none); PART_TYPE Resistor -> (none); SHOWFIELDS YES -> (none); STATUS Released -> (none)
- U1: footprint VFBGA264_14X14_STM -> noob:VFBGA264_14X14_STM
Connections:
- net OTG1_HSDM is gone; now on net USB_DN: U1.A5 (OTG1_HSDM)
- net OTG1_HSDP is gone; now on net USB_DP: U1.B5 (OTG1_HSDP)
- net PE1 is gone; now on net USB_TPD8S_FLT: U1.F17 (PE1)
- net BOOT0: now also R301.1, SW300.2
- net GND: now also C300.2, C301.2, C302.2, C303.2, C304.2, R301.2, R326.2, Y1.2 (G), Y1.4 (G)
- net NRST: now also C304.1, R300.2
- net PWR_ON: now also R304.2
- net at R63.1: now also U1.N14 (PP9)
- net at R57.1: now also U1.J16 (PP3)
- net at R47.1: now also U1.H16 (PP1)
- net at R60.1: now also U1.J15 (PP12)
- net at R64.1: now also U1.L16 (PP8)
- net at R45.1: now also U1.J17 (PP2)
- net at R49.1: now also U1.L15 (PP11)
- net PSRAM_DQS0: now reaches R56.1
- net at R51.1: now also U1.G15 (PP7)
- net OTG1_TXRTUNE: now reaches U1.C6 (OTG1_TXRTUNE)
- net OTG1_TXRTUNE: now also R326.1
- net at R55.1: now also U1.G17 (PP0)
- net at R53.1: now also U1.G16 (PP6)
- net at R46.1: now also U1.L17 (PP14)
- net PSRAM_NCS: now reaches R62.1
- net at R48.1: now also U1.K14 (PP13)
- net at R44.1: now also U1.H15 (PP4)
- net at R61.1: now also U1.H17 (PP15)
- net PSRAM_CLK: now reaches R58.1
- net +1V8_AON: now reaches U1.A1 (PDR_ON)
- net +1V8_AON: now also R304.1
- net PSRAM_DQS1: now reaches R59.1
- net at R50.1: now also U1.N15 (PP10)
- net at R54.1: now also U1.J14 (PP5)
- net CSI_CKN: no longer names the net of U1.U3 (CSI_CKN)
- net CSI_CKP: no longer names the net of U1.T3 (CSI_CKP)
- net CSI_D0N: no longer names the net of U1.U5 (CSI_D0N)
- net CSI_D0P: no longer names the net of U1.T5 (CSI_D0P)
- net CSI_D1N: no longer names the net of U1.U4 (CSI_D1N)
- net CSI_D1P: no longer names the net of U1.T4 (CSI_D1P)
- net PA0 renamed GNSS_PPS
- net PA1 renamed GNSS_EVENT
- net PA10: no longer names the net of U1.R7 (PA10)
- net PA11: no longer names the net of U1.T7 (PA11)
- net PA12: no longer names the net of U1.U7 (PA12)
- net PA13 renamed SWDIO
- net PA14 renamed SWCLK
- net PA15: no longer names the net of U1.P12 (PA15)
- net PA2 renamed USB_VBUS_SENSE
- net PA3 renamed GNSS_RESET_N
- net PA4 renamed GNSS_PVT_STAT
- net PA5 renamed GNSS_RTK_STAT
- net PA6 renamed DEV_BOOT
- net PA7 renamed GNSS_ERR_STAT
- net PA8: no longer names the net of U1.U8 (PA8)
- net PA9: no longer names the net of U1.P7 (PA9)
- net PB0 renamed IMU_DRY_SYNC
- net PB1 renamed IMU_RESET_N
- net PB10 renamed ESP_UART_TX
- net PB11 renamed ESP_UART_RX
- net PB12: no longer names the net of U1.R10 (PB12)
- net PB13: no longer names the net of U1.C15 (PB13)
- net PB14: no longer names the net of U1.B17 (PB14)
- net PB15: no longer names the net of U1.D17 (PB15)
- net PB2: no longer names the net of U1.C16 (PB2)
- net PB3: no longer names the net of U1.F13 (PB3)
- net PB4: no longer names the net of U1.T12 (PB4)
- net PB5 renamed SWO
- net PB6: no longer names the net of U1.E17 (PB6)
- net PB7: no longer names the net of U1.E16 (PB7)
- net PB8: no longer names the net of U1.D16 (PB8)
- net PB9: no longer names the net of U1.D15 (PB9)
- net PC0: no longer names the net of U1.C10 (PC0)
- net PC1: no longer names the net of U1.A9 (PC1)
- net PC10 renamed SD_D2
- net PC11 renamed SD_D3
- net PC12 renamed SD_CLK
- net PC13: no longer names the net of U1.F3 (PC13)
- net PC14 renamed LSE_IN
- net LSE_IN: now also C302.1, Y2.1
- net PC15 renamed LSE_OUT
- net LSE_OUT: now also C303.1, Y2.2
- net PC2: no longer names the net of U1.D9 (PC2)
- net PC3: no longer names the net of U1.E10 (PC3)
- net PC4 renamed ESP_UART_CTS
- net PC5: no longer names the net of U1.B10 (PC5)
- net PC6 renamed GNSS_UART_TX
- net PC7 renamed GNSS_UART_RX
- net PC8 renamed SD_D0
- net PC9 renamed SD_D1
- net PD0 renamed ESP_EN
- net PD1 renamed ESP_BOOT
- net PD10 renamed LED_RUN
- net PD11 renamed LED_WARN
- net PD12 renamed LED_ERR
- net PD13: no longer names the net of U1.C17 (PD13)
- net PD14 renamed PMIC_SCL
- net PD15 renamed PMIC_SDA
- net PD2: no longer names the net of U1.C12 (PD2)
- net PD3 renamed ESP_HOST_WAKE
- net PD4: no longer names the net of U1.B15 (PD4)
- net PD5: no longer names the net of U1.D14 (PD5)
- net PD6: no longer names the net of U1.D12 (PD6)
- net PD7: no longer names the net of U1.E12 (PD7)
- net PD8: no longer names the net of U1.E14 (PD8)
- net PD9: no longer names the net of U1.H14 (PD9)
- net PE0 renamed BUCK_3V3_PG
- net PE10 renamed AUX5_EN
- net PE11: no longer names the net of U1.E11 (PE11)
- net PE12: no longer names the net of U1.B12 (PE12)
- net PE13: no longer names the net of U1.A11 (PE13)
- net PE14: no longer names the net of U1.B11 (PE14)
- net PE15: no longer names the net of U1.A12 (PE15)
- net PE2 renamed BAT_ALRT
- net PE3 renamed CHG_INT
- net PE4 renamed USBPD_INT
- net PE5 renamed USBPD_SCL
- net PE6 renamed USBPD_SDA
- net PE7 renamed RADIO_EN
- net PE8 renamed GNSS_EN
- net PE9 renamed IMU_EN
- net PF0: no longer names the net of U1.R3 (PF0)
- net PF1: no longer names the net of U1.P4 (PF1)
- net PF10: no longer names the net of U1.L4 (PF10)
- net PF11: no longer names the net of U1.P3 (PF11)
- net PF12: no longer names the net of U1.T1 (PF12)
- net PF13: no longer names the net of U1.R2 (PF13)
- net PF14: no longer names the net of U1.N2 (PF14)
- net PF15: no longer names the net of U1.N1 (PF15)
- net PF2: no longer names the net of U1.N4 (PF2)
- net PF3: no longer names the net of U1.M2 (PF3)
- net PF4: no longer names the net of U1.L2 (PF4)
- net PF5: no longer names the net of U1.M3 (PF5)
- net PF6: no longer names the net of U1.L5 (PF6)
- net PF7: no longer names the net of U1.M1 (PF7)
- net PF8: no longer names the net of U1.N3 (PF8)
- net PF9: no longer names the net of U1.P1 (PF9)
- net PG0: no longer names the net of U1.R13 (PG0)
- net PG1: no longer names the net of U1.R9 (PG1)
- net PG10 renamed ESP_UART_RTS
- net PG11: no longer names the net of U1.U13 (PG11)
- net PG12: no longer names the net of U1.T9 (PG12)
- net PG13: no longer names the net of U1.U9 (PG13)
- net PG14: no longer names the net of U1.P6 (PG14)
- net PG15: no longer names the net of U1.R6 (PG15)
- net PG2: no longer names the net of U1.T11 (PG2)
- net PG3: no longer names the net of U1.R1 (PG3)
- net PG4: no longer names the net of U1.P2 (PG4)
- net PG5: no longer names the net of U1.M4 (PG5)
- net PG6: no longer names the net of U1.L3 (PG6)
- net PG7: no longer names the net of U1.L1 (PG7)
- net PG8: no longer names the net of U1.T14 (PG8)
- net PG9: no longer names the net of U1.T13 (PG9)
- net PH0 renamed HSE_IN
- net HSE_IN: now also C300.1, Y1.1
- net PH1 renamed HSE_OUT
- net HSE_OUT: now also C301.1, Y1.3
- net PH2 renamed SD_CMD
- net PH3 renamed SD_CD_N
- net PH4: no longer names the net of U1.F4 (PH4)
- net PH5 renamed IMU_SPI_SCK
- net PH6 renamed IMU_SPI_CS_N
- net PH7 renamed IMU_SPI_MOSI
- net PH8 renamed IMU_SPI_MISO
- net PH9: no longer names the net of U1.D8 (PH9)
- net PN0: no longer names the net of U1.P17 (PN0)
- net PN1: no longer names the net of U1.R17 (PN1)
- net PN1: now also R325.2
- net PN10: no longer names the net of U1.U15 (PN10)
- net PN11: no longer names the net of U1.U16 (PN11)
- net PN12: no longer names the net of U1.P14 (PN12)
- net PN2: no longer names the net of U1.T17 (PN2)
- net PN2: now also R320.2
- net PN3: no longer names the net of U1.R15 (PN3)
- net PN3: now also R321.2
- net PN4: no longer names the net of U1.N17 (PN4)
- net PN4: now also R322.2
- net PN5: no longer names the net of U1.R16 (PN5)
- net PN5: now also R323.2
- net PN6: no longer names the net of U1.P15 (PN6)
- net PN6: now also R324.2
- net PN7: no longer names the net of U1.T16 (PN7)
- net PN8: no longer names the net of U1.P16 (PN8)
- net PN9: no longer names the net of U1.T15 (PN9)
- net PO0: no longer names the net of R62.2, U1.M17 (PO0)
- net PO1: no longer names the net of U1.K16 (PO1)
- net PO2: no longer names the net of R56.2, U1.K17 (PO2)
- net PO3: no longer names the net of R59.2, U1.M16 (PO3)
- net PO4: no longer names the net of R58.2, U1.N16 (PO4)
- net PO5: no longer names the net of U1.K15 (PO5)
- net PP0 renamed PSRAM_IO0
- net PSRAM_IO0: no longer U1.G17 (PP0)
- net PP1 renamed PSRAM_IO1
- net PSRAM_IO1: no longer U1.H16 (PP1)
- net PP10 renamed PSRAM_IO10
- net PSRAM_IO10: no longer U1.N15 (PP10)
- net PP11 renamed PSRAM_IO11
- net PSRAM_IO11: no longer U1.L15 (PP11)
- net PP12 renamed PSRAM_IO12
- net PSRAM_IO12: no longer U1.J15 (PP12)
- net PP13 renamed PSRAM_IO13
- net PSRAM_IO13: no longer U1.K14 (PP13)
- net PP14 renamed PSRAM_IO14
- net PSRAM_IO14: no longer U1.L17 (PP14)
- net PP15 renamed PSRAM_IO15
- net PSRAM_IO15: no longer U1.H17 (PP15)
- net PP2 renamed PSRAM_IO2
- net PSRAM_IO2: no longer U1.J17 (PP2)
- net PP3 renamed PSRAM_IO3
- net PSRAM_IO3: no longer U1.J16 (PP3)
- net PP4 renamed PSRAM_IO4
- net PSRAM_IO4: no longer U1.H15 (PP4)
- net PP5 renamed PSRAM_IO5
- net PSRAM_IO5: no longer U1.J14 (PP5)
- net PP6 renamed PSRAM_IO6
- net PSRAM_IO6: no longer U1.G16 (PP6)
- net PP7 renamed PSRAM_IO7
- net PSRAM_IO7: no longer U1.G15 (PP7)
- net PP8 renamed PSRAM_IO8
- net PSRAM_IO8: no longer U1.L16 (PP8)
- net PP9 renamed PSRAM_IO9
- net PSRAM_IO9: no longer U1.N14 (PP9)
- net PQ0 renamed BTN1_N
- net PQ1 renamed BTN2_N
- net PQ2 renamed BTN3_N
- net PQ3: no longer names the net of U1.D3 (PQ3)
- net PQ4: no longer names the net of U1.D4 (PQ4)
- net PQ5: no longer names the net of U1.D5 (PQ5)
- net PQ6: no longer names the net of U1.A2 (PQ6)
- net PQ7: no longer names the net of U1.G5 (PQ7)
- net UCPD1_CC1: no longer names the net of U1.A6 (UCPD1_CC1)
- net UCPD1_CC2: no longer names the net of U1.B6 (UCPD1_CC2)
- new net +3V3_MAIN: R300.1, SW300.1
- new net FLASH_CLK: R324.1
- new net FLASH_IO0: R320.1
- new net FLASH_IO1: R321.1
- new net FLASH_IO2: R322.1
- new net FLASH_IO3: R323.1
- new net FLASH_NCS: R325.1
- no-connect marks 6 -> 99
Other:
- note added: "OTG1_TXRTUNE: R326 = 200 ohm +/-1% to GND; place close to the USB PHY1 pin."
- note added: "USB_VBUS_SENSE is about 0.507 V when AP_V5V is 5 V; use a long ADC sampling time."
