File: pcb/v2_pcb/STM32_MCU_IO.kicad_sch (KiCad schematic)
At the start: 39 parts, among them SW300 BOOT, U1 STM32N657X0H3Q, Y1 NX2016SA-24MHZ-EXS00A-CS10820, Y2 NX2012SA-32.768KHZ-EXS00A-MU0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

Commit message: minor fixes
Parts:
- C300, C301, C302, C303: value 8.2pF C0G (TUNE) -> 8.2pF 50V C0G (TUNE); Dielectric (none) -> C0G; MPN (none) -> GCQ1555C1H8R2BB01D; Manufacturer (none) -> Murata; Qualification (none) -> AEC-Q200; Release_Status (none) -> TUNE - validate oscillation margin and frequency on final P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; Tolerance (none) -> ±0.1 pF; Voltage (none) -> 50 VDC
- C304: value 100nF -> 10nF 50V X7R; Design_Note (none) -> STM32N6 NRST capacitor; keep at or below ST 10 nF maximum; Dielectric (none) -> X7R; MPN (none) -> CGA2B3X7R1H103K050BE; Manufacturer (none) -> TDK; Qualification (none) -> AEC-Q200; Termination (none) -> Soft termination; Tolerance (none) -> ±10%; Voltage (none) -> 50 VDC
- R300, R301: MPN (none) -> CRCW040210K0FKED; Manufacturer (none) -> Vishay; Power (none) -> 0.063 W; TCR (none) -> ±100 ppm/K; Tolerance (none) -> ±1%
- R304: MPN (none) -> CRCW0402100KFKED; Manufacturer (none) -> Vishay; Power (none) -> 0.063 W; TCR (none) -> ±100 ppm/K; Tolerance (none) -> ±1%
- R320, R321, R322, R323, R324, R325, R44, R45, R46, R47, R48, R49, R50, R51, R53, R54, R55, R56, R57, R58, R59, R60, R61, R62, R63, R64: MPN RC0402FR-0722RL -> CRCW040222R0FKED; Manufacturer Yageo -> Vishay; Power (none) -> 0.063 W; Qualification (none) -> AEC-Q200; TCR (none) -> ±100 ppm/K; Tolerance (none) -> ±1%
- R326: MPN RC0402FR-07200RL -> CRCW0402200RFKED; Manufacturer Yageo -> Vishay; Power (none) -> 0.063 W; Qualification (none) -> AEC-Q200; TCR (none) -> ±100 ppm/K; Tolerance (none) -> ±1%
- SW300: value BOOT -> KMR223NG ULC LFG; Contact (none) -> Gold ULC; 1 µA minimum at 1.8 V; MPN KMR221GLFS -> Y78B22324FP; Manufacturer C&K -> Littelfuse (C&K); Operating_Temperature (none) -> -40 to +125 °C
- U1: Design_Note (none) -> Program OTP124 mask 0x00018000 (VDDIO2/VDDIO3 1.8 V selecti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; MPN (none) -> STM32N657X0H3Q; Manufacturer (none) -> STMicroelectronics
Connections:
- net ESP_UART_RTS: now also U1.M3 (PF5); no longer U1.T10 (PG10)
Other:
- note added: "BOOT-ROM PIN CONFLICT AVOIDED: ESP_UART_RTS is PF5 / ball M3; PG10 / ball T10 remains free for ROM USART5_TX."
- note added: "PROVISIONING: program OTP124 mask 0x00018000 so VDDIO2/VDDIO3 are 1.8 V before enabling attached interfaces; verify readback in production."

Commit message: remove resistors on flash line
Parts:
- removed R320, R321, R322, R323, R324, R325, R44, R45, R46, R47, R48, R49, R50, R51, R53, R54, R55, R56, R57, R59, R60, R61, R62, R63, R64: 22R, Resistor_SMD:R_0402_1005Metric, symbol Device:R_Small_US
Connections:
- net FLASH_CLK: now also U1.P15 (PN6)
- net FLASH_IO0: now also U1.T17 (PN2)
- net FLASH_IO1: now also U1.R15 (PN3)
- net FLASH_IO2: now also U1.N17 (PN4)
- net FLASH_IO3: now also U1.R16 (PN5)
- net FLASH_NCS: now also U1.R17 (PN1)
- net PSRAM_DQS0: now also U1.K17 (PO2)
- net PSRAM_DQS1: now also U1.M16 (PO3)
- net PSRAM_IO0: now also U1.G17 (PP0)
- net PSRAM_IO1: now also U1.H16 (PP1)
- net PSRAM_IO10: now also U1.N15 (PP10)
- net PSRAM_IO11: now also U1.L15 (PP11)
- net PSRAM_IO12: now also U1.J15 (PP12)
- net PSRAM_IO13: now also U1.K14 (PP13)
- net PSRAM_IO14: now also U1.L17 (PP14)
- net PSRAM_IO15: now also U1.H17 (PP15)
- net PSRAM_IO2: now also U1.J17 (PP2)
- net PSRAM_IO3: now also U1.J16 (PP3)
- net PSRAM_IO4: now also U1.H15 (PP4)
- net PSRAM_IO5: now also U1.J14 (PP5)
- net PSRAM_IO6: now also U1.G16 (PP6)
- net PSRAM_IO7: now also U1.G15 (PP7)
- net PSRAM_IO8: now also U1.L16 (PP8)
- net PSRAM_IO9: now also U1.N14 (PP9)
- net PSRAM_NCS: now also U1.M17 (PO0)

Commit message: swithc 3to 3 layer signal for ram
Changed lines of the file:
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@@
 		)
+	)
+	(junction
+		(at 299.72 207.01)
+		(diameter 0)
+		(color 0 0 0 0)
 	)
 	(no_connect
