File: pcb/v2_pcb/Power.kicad_sch (KiCad schematic)
At the start: 112 parts, among them J20 2S_PACK_BALANCE, Q3 NMOS, Q4 NMOS, Q5 NMOS, U10 TPSM863253RDXR, U11 TPS22997RYZR, U20 TPS630701RNMR (5V fixed), U21 TPS22918DBVR, U22 TPS22918DBVR, U23 TPS22918DBVR, U6 BQ25798RQMR, U7 MAX17320G22+, U8 RPL-3.0-R

Commit message: minor fixes
Parts:
- added C18: 10nF 50V X7R, Capacitor_SMD:C_0603_1608Metric, symbol Device:C_Small
- added R20: 100R 1%, Resistor_SMD:R_0603_1608Metric, symbol Device:R_Small_US
- C10, C233, C234, C42, C56, C62, C81, C82, C84, C85, C87, C88, C9, C91, C93: value 10uF 25V X7R -> 10uF 50V X7R; Dielectric (none) -> X7R; MPN (none) -> CNA6P1X7R1H106K250AE; Manufacturer (none) -> TDK; Qualification (none) -> AEC-Q200; Termination (none) -> Soft termination / low resistance; Tolerance (none) -> ±10%; Voltage (none) -> 50 VDC
- C11, C14, C187, C7, C83, C86: value 100nF 25V X7R -> 100nF 50V X7R; Dielectric (none) -> X7R; MPN (none) -> CGA3E2X7R1H104K080AE; Manufacturer (none) -> TDK; Qualification (none) -> AEC-Q200; Termination (none) -> Soft termination; Tolerance (none) -> ±10%; Voltage (none) -> 50 VDC
- C12, C8: value 10nF 25V X7R -> 10nF 50V X7R; Dielectric (none) -> X7R; MPN (none) -> CGA3E2X7R1H103K080AE; Manufacturer (none) -> TDK; Qualification (none) -> AEC-Q200; Termination (none) -> Soft termination; Tolerance (none) -> ±10%; Voltage (none) -> 50 VDC
- C13: value 100nF 25V X7R -> 470nF 25V X7R; Dielectric (none) -> X7R; MPN (none) -> CGA3E3X7R1E474K080AE; Manufacturer (none) -> TDK; Qualification (none) -> AEC-Q200; Termination (none) -> Soft termination; Tolerance (none) -> ±10%; Voltage (none) -> 25 VDC
- C15, C16, C17: value 470nF 10V X7R -> 470nF 25V X7R; Dielectric (none) -> X7R; MPN (none) -> CGA3E3X7R1E474K080AE; Manufacturer (none) -> TDK; Qualification (none) -> AEC-Q200; Termination (none) -> Soft termination; Tolerance (none) -> ±10%; Voltage (none) -> 25 VDC
- C180: Dielectric (none) -> X7R; MPN (none) -> CGA5L1X7R1E106K160AE; Manufacturer (none) -> TDK; Qualification (none) -> AEC-Q200; Termination (none) -> Soft termination; Tolerance (none) -> ±10%; Voltage (none) -> 25 VDC
- C181, C188, C189: Dielectric (none) -> X7R; MPN (none) -> GCJ31CR71A226KE01L; Manufacturer (none) -> Murata; Qualification (none) -> AEC-Q200; Termination (none) -> Soft termination; Tolerance (none) -> ±10%; Voltage (none) -> 10 VDC
- C182: value 22pF C0G -> 22pF 50V C0G; Dielectric (none) -> C0G; MPN (none) -> CGA3E2C0G1H220J080AA; Manufacturer (none) -> TDK; Qualification (none) -> AEC-Q200; Tolerance (none) -> ±5%; Voltage (none) -> 50 VDC
- C186: footprint Capacitor_SMD:C_1206_3216Metric -> Capacitor_SMD:C_1210_3225Metric; Dielectric (none) -> X7R; MPN (none) -> CGA6P3X7R1E226M250AE; Manufacturer (none) -> TDK; Qualification (none) -> AEC-Q200; Release_Status (none) -> Verify >10uF effective at VSYS_RAW,max including bias, tole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; Termination (none) -> Soft termination; Tolerance (none) -> ±20%; Voltage (none) -> 25 VDC
- C190, C240: value 100nF 10V X7R -> 100nF 50V X7R; Dielectric (none) -> X7R; MPN (none) -> CGA3E2X7R1H104K080AE; Manufacturer (none) -> TDK; Qualification (none) -> AEC-Q200; Termination (none) -> Soft termination; Tolerance (none) -> ±10%; Voltage (none) -> 50 VDC
- C191, C244: value 1uF 10V X7R -> 1uF 25V X7R; Dielectric (none) -> X7R; MPN (none) -> CGA3E1X7R1E105K080AE; Manufacturer (none) -> TDK; Qualification (none) -> AEC-Q200; Termination (none) -> Soft termination; Tolerance (none) -> ±10%; Voltage (none) -> 25 VDC
- C192: value 3.9nF 50V C0G -> 3.9nF 100V C0G; Dielectric (none) -> C0G; MPN (none) -> CGA3E1C0G2A392J080AE; Manufacturer (none) -> TDK; Qualification (none) -> AEC-Q200; Termination (none) -> Soft termination; Tolerance (none) -> ±5%; Voltage (none) -> 100 VDC
- C235, C239: value 10uF 25V X5R -> 10uF 25V X7S; footprint Capacitor_SMD:C_0603_1608Metric -> Capacitor_SMD:C_0805_2012Metric; Dielectric (none) -> X7S; MPN (none) -> GCJ21BC71E106KE02L; Manufacturer (none) -> Murata; Qualification (none) -> AEC-Q200; Release_Status (none) -> Supplemental capacitance; verify effective C under worst-ca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; Termination (none) -> Soft termination; Tolerance (none) -> ±10%; Voltage (none) -> 25 VDC
- C236, C237, C238: value 22uF 10V X7R -> 22uF 25V X7R; Dielectric (none) -> X7R; MPN (none) -> CGA6P3X7R1E226M250AE; Manufacturer (none) -> TDK; Qualification (none) -> AEC-Q200; Termination (none) -> Soft termination; Tolerance (none) -> ±20%; Voltage (none) -> 25 VDC
- C241, C242, C243: value 1nF C0G -> 1nF 100V C0G; Dielectric (none) -> C0G; MPN (none) -> CGA3E2C0G2A102J080AE; Manufacturer (none) -> TDK; Qualification (none) -> AEC-Q200; Termination (none) -> Soft termination; Tolerance (none) -> ±5%; Voltage (none) -> 100 VDC
- C245, C248: Dielectric (none) -> X7R; MPN (none) -> GCJ21BR71A106KE01L; Manufacturer (none) -> Murata; Qualification (none) -> AEC-Q200; Termination (none) -> Soft termination; Tolerance (none) -> ±10%; Voltage (none) -> 10 VDC
- C246, C249, C252: value 100nF -> 100nF 50V X7R; Dielectric (none) -> X7R; MPN (none) -> CGA3E2X7R1H104K080AE; Manufacturer (none) -> TDK; Qualification (none) -> AEC-Q200; Termination (none) -> Soft termination; Tolerance (none) -> ±10%; Voltage (none) -> 50 VDC
- C247, C250: value 1uF 10V X7R -> 1uF 50V X7R; Dielectric (none) -> X7R; MPN (none) -> CGA4J3X7R1H105K125AE; Manufacturer (none) -> TDK; Qualification (none) -> AEC-Q200; Termination (none) -> Soft termination; Tolerance (none) -> ±10%; Voltage (none) -> 50 VDC
- C251, C92: value 4.7uF 10V X7R -> 4.7uF 16V X7R; Dielectric (none) -> X7R; MPN (none) -> CGA4J3X7R1C475K125AE; Manufacturer (none) -> TDK; Qualification (none) -> AEC-Q200; Termination (none) -> Soft termination; Tolerance (none) -> ±10%; Voltage (none) -> 16 VDC
- C49, C53: value 47nF 16V X7R -> 47nF 50V X7R; Dielectric (none) -> X7R; MPN (none) -> CGA3E2X7R1H473K080AE; Manufacturer (none) -> TDK; Qualification (none) -> AEC-Q200; Termination (none) -> Soft termination; Tolerance (none) -> ±10%; Voltage (none) -> 50 VDC
- D2: value LTST-C190KGKT GREEN -> ASMT-RF45-AN002 YELLOW GREEN; Color (none) -> Yellow green; Current (none) -> 20 mA maximum; visual-qualify at fitted 1 kΩ drive; MPN LTST-C190KGKT -> ASMT-RF45-AN002; Manufacturer (none) -> Broadcom; Operating_Temperature (none) -> -40 to +100 °C; Qualification (none) -> Automotive qualified
- F1: value 5A hold / 24V PTC -> 5.0A Ihold @23C / 24V PTC; Design_Note (none) -> HOLD: Ihold derates to 4.25 A at 40 C and 3.25 A at 60 C; d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; MPN 2920L500/24DR -> 2920L500/24SLDR; Qualification_Status (none) -> UNRESOLVED_THERMAL_CURRENT_BUDGET
- FB20, FB21: value 600R@100MHz 1A -> 600Ω @ 100MHz, 1.4A AEC-Q200; footprint Inductor_SMD:L_0805_2012Metric -> open-race-v2:FB_Murata_BLM21_2.0x1.25mm; Current (none) -> 1.4 A to 85 °C; 0.9 A at 125 °C; DCR (none) -> ≤0.14 Ω initial; Impedance (none) -> 600 Ω ±25% @ 100 MHz; MPN BLM21PG601SN1D -> BLM21PG601SH1D; Operating_Temperature (none) -> -55 to +125 °C; Qualification (none) -> AEC-Q200; automotive powertrain/safety
- L1: value 2.2uH XAL7030-222ME -> 2.2uH XAL7030-222MEC; MPN XAL7030-222ME -> XAL7030-222MEC; Manufacturer (none) -> Coilcraft
- L20: value 1.5uH XFL4020-152ME -> 1.5uH XFL4020-152MEC
- NTC1: Manufacturer (none) -> Murata
- Q3, Q4, Q5: value NMOS -> CSD18540Q5B
- R10: MPN (none) -> CRCW060310R0FKEA; Manufacturer (none) -> Vishay; Power (none) -> 0.10 W; TCR (none) -> ±100 ppm/K; Tolerance (none) -> ±1%
- R11, R12: footprint Resistor_SMD:R_0603_1608Metric -> Resistor_SMD:R_1206_3216Metric; MPN (none) -> CRCW120668R0FKEAHP; Manufacturer (none) -> Vishay; Power (none) -> 0.75 W; TCR (none) -> ±100 ppm/K; Tolerance (none) -> ±1%
- R13: Manufacturer (none) -> Vishay Dale; Power (none) -> 1.0 W at 70 °C; Qualification (none) -> AEC-Q200; TCR (none) -> ±75 ppm/K; Tolerance (none) -> ±1%
- R221, R24, R240, R29, R30, R31, R37, R38, R39: MPN (none) -> CRCW060310K0FKEA; Manufacturer (none) -> Vishay; Power (none) -> 0.10 W; TCR (none) -> ±100 ppm/K; Tolerance (none) -> ±1%
- R222, R6, R9: MPN (none) -> CRCW06031K00FKEA; Manufacturer (none) -> Vishay; Power (none) -> 0.10 W; TCR (none) -> ±100 ppm/K; Tolerance (none) -> ±1%
- R223: MPN (none) -> CRCW060347K0FKEA; Manufacturer (none) -> Vishay; Power (none) -> 0.10 W; TCR (none) -> ±100 ppm/K; Tolerance (none) -> ±1%
- R224: MPN (none) -> CRCW060337K4FKEA; Manufacturer (none) -> Vishay; Power (none) -> 0.10 W; TCR (none) -> ±100 ppm/K; Tolerance (none) -> ±1%
- R228: MPN (none) -> CRCW0603220KFKEA; Manufacturer (none) -> Vishay; Power (none) -> 0.10 W; TCR (none) -> ±100 ppm/K; Tolerance (none) -> ±1%
- R229, R244, R245, R246, R247, R248: MPN (none) -> CRCW0603100KFKEA; Manufacturer (none) -> Vishay; Power (none) -> 0.10 W; TCR (none) -> ±100 ppm/K; Tolerance (none) -> ±1%
- R23, R7, R8: MPN (none) -> CRCW0603100RFKEA; Manufacturer (none) -> Vishay; Power (none) -> 0.10 W; TCR (none) -> ±100 ppm/K; Tolerance (none) -> ±1%
- R25: value 5.24k 1% -> 5.23k 1%; MPN (none) -> CRCW06035K23FKEA; Manufacturer (none) -> Vishay; Power (none) -> 0.10 W; TCR (none) -> ±100 ppm/K; Tolerance (none) -> ±1%
- R26: value 30.3k 1% -> 30.1k 1%; MPN (none) -> CRCW060330K1FKEA; Manufacturer (none) -> Vishay; Power (none) -> 0.10 W; TCR (none) -> ±100 ppm/K; Tolerance (none) -> ±1%
- R28: MPN (none) -> CRCW06032K20FKEA; Manufacturer (none) -> Vishay; Power (none) -> 0.10 W; TCR (none) -> ±100 ppm/K; Tolerance (none) -> ±1%
- R35: MPN (none) -> CRCW06038K20FKEA; Manufacturer (none) -> Vishay; Power (none) -> 0.10 W; TCR (none) -> ±100 ppm/K; Tolerance (none) -> ±1%
- TP1, TP20: now left out of the parts list
- U10: footprint Package_DFN_QFN:Texas_RDX0007A_QFN-FCMOD-7-3.3x4mm-P0.5mm_4EP -> open-race-v2:Texas_RDX0007A_QFN-FCMOD-7-3.3x4mm-P0.5mm_4EP_NoVias; Footprint rationale (none) -> TI RDX0007A optional 0.20 mm under-pad vias omitted; add fa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
- U6: MPN (none) -> BQ25798RQMR; Manufacturer (none) -> Texas Instruments
- U7: Manufacturer (none) -> Analog Devices (Maxim Integrated)
Connections:
- net GND1: now also C18.2
- net PACK_POS: no longer F1.1, J20.1 (Pin_1)
- net PACK_POS_CONN: now also F1.1, J20.1 (Pin_1)
- net vpack+: now also Q5.1 (S), Q5.2 (S), Q5.3 (S)
- net at Q5.4 (G): now also R8.1
- net at Q5.5 (D), Q5.6 (D), Q5.7 (D)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: now also Q4.5 (D), Q4.6 (D), Q4.7 (D), Q4.8 (D)
- net at R6.2, U7.6 (PCKP): now also C18.1
- net at Q3.4 (G): now also R20.2; no longer U6.24 (SDRV)
- new net: R20.1, U6.24 (SDRV)
Other:
- note added: "5 V AUX BUCK-BOOST — TPS630701RNMR"
- note added: "POWER TREE — REGULATOR STAGES VSYS_RAW -> U10 (3.3 V) -> +3V3_MAIN; open-drain PG drives BUCK_3V3_PG. VSYS_RAW -> U8 (1.8 V) -> +1V8_AON; CTRL = BUCK_3V3_PG with +3V3_MAIN pull-up. VSYS_RAW -> U20 (fixed 5 V buck-boost) -> +5V_AUX; AUX5_EN controls EN. Validate all rails across the approved loaded 2S operating range and transient cases. +1V8_AON -> U11 (PWR_ON enabled) -> +1V8_RUN."
- note removed: "5 V AUX BUCK — RPL-3.0-R"
- note removed: "POWER TREE — BUCK STAGES ADDED VSYS_RAW -> U10 (3.3 V) -> +3V3_MAIN; open-drain PG drives BUCK_3V3_PG. VSYS_RAW -> U8 (1.8 V) -> +1V8_AON; CTRL = BUCK_3V3_PG with +3V3_MAIN pull-up. VSYS_RAW -> U9 (5 V) -> +5V_AUX; CTRL tied to VIN. WARNING: the 5 V buck needs about 6.8 V input to regulate; validate the loaded 2S minimum. +1V8_AON -> U11 (PWR_ON enabled) -> +1V8_RUN."
- moved on the sheet: Q5
