File: pcb/v2_pcb/open-race_v2.kicad_sch (KiCad schematic)
At the start: 0 parts

Commit message: minor fixes
Other:
- sheet STM32 MCU I/O renamed STM32 MCU IO
Changed lines of the file:
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@@
 	(bus
 		(pts
-			(xy 107.95 66.04) (xy 186.69 66.04)
+			(xy 109.22 66.04) (xy 124.46 66.04)
 		)
 		(stroke
@@
 	(bus
 		(pts
-			(xy 107.95 66.04) (xy 107.95 210.82)
+			(xy 186.69 66.04) (xy 190.5 66.04)
+		)
+		(stroke
+			(width 0)
+			(type default)
+		)
+	)
+	(bus
+		(pts
+			(xy 190.5 66.04) (xy 190.5 72.39)
+		)
+		(stroke
+			(width 0)
+			(type default)
+		)
+	)
+	(bus
+		(pts
+			(xy 190.5 72.39) (xy 107.95 72.39)
+		)
+		(stroke
+			(width 0)
+			(type default)
+		)
+	)
+	(bus
+		(pts
+			(xy 107.95 72.39) (xy 107.95 210.82)
 		)
 		(stroke
@@
 			(color 0 0 0 0)
 		)
-		(property "Sheetname" "STM32 MCU I/O"
+		(property "Sheetname" "STM32 MCU IO"
 			(at 124.46 41.1984 0)
 			(show_name no)
