File: pcb/v2_pcb/open-race_v2.kicad_pcb (KiCad board)
At the start: 8 copper layers, 90.5 x 49.5 mm, 356 parts, among them IC1 AP33772SDKZ-13-FA01, J1 Conn_ARM_SWD_TagConnect_TC203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, J2 USB4105-GF-A, J20 2S_PACK_BALANCE, J3 DM3CS-SF, J800 ESP UART PROGRAM (pin 1 VTREF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, J900 U.FL / Beitian BT-T076, Q1 NMOS, Q2 NMOS, Q3 NMOS, Q4 NMOS, Q5 NMOS, SW1101 BUTTON 1, SW1102 BUTTON 2, SW1103 BUTTON 3, SW300 BOOT, SW301 DEV BOOT, SW800 RESET, SW801 BOOT, U1 STM32N657X0H3Q, U10 TPSM863253RDXR, U1000 SCH16T-K01, U11 TPS22997RYZR, U1100 SN74AHCT1G125DCKR, U1101 SN74AHCT1G125DCKR, U20 TPS630701RNMR (5V fixed), U21 TPS22918DBVR, U22 TPS22918DBVR, U23 TPS22918DBVR, U24 TXS0104EPW, U25 TPS3808G01DBVR, U3 APS512XXN-OB9-BG, U4 TPD8S300ARUKR, U5 MX25U51279GXDR00, U6 BQ25798RQMR, U7 MAX17320G22+, U8 RPL-3.0-R, U800 ESP32-C6-MINI-1, U900 UM980, Y1 NX2016SA-24MHZ-EXS00A-CS10820, Y2 NX2012SA-32.768KHZ-EXS00A-MU0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

Commit message: minor fixes
Parts:
- removed C305: 100nF, Capacitor_SMD:C_0402_1005Metric
- added C18: 10nF 50V X7R, Capacitor_SMD:C_0603_1608Metric, F.Cu at (190.0, 100.0)
- added C255: 1uF 25V X7R, Capacitor_SMD:C_0603_1608Metric, F.Cu at (200.0, 100.0)
- added C256: 1uF 25V X7R, Capacitor_SMD:C_0603_1608Metric, F.Cu at (205.0, 100.0)
- added D3: TVS2200DRVR, open-race-v2:WSON-6-1EP_2x2mm_P0.65mm_EP1x1.6mm_TVS2200, F.Cu at (220.0, 100.0)
- added R174: 10.0k 1%, Resistor_SMD:R_0402_1005Metric, F.Cu at (215.0, 100.0)
- added R20: 100R 1%, Resistor_SMD:R_0603_1608Metric, F.Cu at (195.0, 100.0)
- added U26: TLV75533PDBVR, Package_TO_SOT_SMD:SOT-23-5, F.Cu at (210.0, 100.0)
- C1, C1002, C1004, C1100, C1101, C1110, C1111, C1112, C1113, C1114, C1121, C1122, C1123, C141, C142, C169, C2, C231, C232, C246, C249, C252, C28, C306, C309, C36, C39, C4, C40, C46, C47, C48, C50, C52, C54, C55, C58, C59, C64, C66, C67, C71, C72, C73, C74, C75, C76, C77, C78, C79, C80, C801, C89, C901, C904: value 100nF -> 100nF 50V X7R
- C10, C233, C234, C42, C56, C62, C81, C82, C84, C85, C87, C88, C9, C91, C93: value 10uF 25V X7R -> 10uF 50V X7R
- C1000, C1003, C143, C800: value 1uF -> 1uF 25V X7R
- C1001, C29, C307, C35, C802, C903: value 10uF -> 10uF 10V X7R
- C11, C14, C187, C7, C83, C86: value 100nF 25V X7R -> 100nF 50V X7R
- C1115, C803: value 47uF -> 47uF 10V X7R; footprint Capacitor_SMD:C_0805_2012Metric -> Capacitor_SMD:C_1210_3225Metric
- C12, C8: value 10nF 25V X7R -> 10nF 50V X7R
- C13: value 100nF 25V X7R -> 470nF 25V X7R
- C144, C34, C90: value 4.7uF -> 4.7uF 16V X7S
- C15, C16, C17: value 470nF 10V X7R -> 470nF 25V X7R
- C170, C176, C177, C178, C179, C905, C906: value 22uF -> 22uF 6.3V X7T
- C182: value 22pF C0G -> 22pF 50V C0G
- C186: footprint Capacitor_SMD:C_1206_3216Metric -> Capacitor_SMD:C_1210_3225Metric
- C190, C240, C253: value 100nF 10V X7R -> 100nF 50V X7R
- C191, C244: value 1uF 10V X7R -> 1uF 25V X7R
- C192: value 3.9nF 50V C0G -> 3.9nF 100V C0G
- C230: value 1uF 35V X7R -> 1uF 50V X7R
- C235, C239: value 10uF 25V X5R -> 10uF 25V X7S; footprint Capacitor_SMD:C_0603_1608Metric -> Capacitor_SMD:C_0805_2012Metric
- C236, C237, C238: value 22uF 10V X7R -> 22uF 25V X7R
- C241, C242, C243: value 1nF C0G -> 1nF 100V C0G
- C247, C250, C3, C6: value 1uF 10V X7R -> 1uF 50V X7R
- C251, C92: value 4.7uF 10V X7R -> 4.7uF 16V X7R
- C254: value 1nF 10V X7R -> 1nF 100V C0G
- C300, C301, C302, C303: value 8.2pF C0G (TUNE) -> 8.2pF 50V C0G (TUNE)
- C304: value 100nF -> 10nF 50V X7R
- C308, C38, C41, C43, C44, C45, C51, C57, C60, C61, C63, C65, C68, C69, C70: value 1uF -> 1uF 10V X7S
- C49, C53: value 47nF 16V X7R -> 47nF 50V X7R
- C900, C902: value 100pF C0G -> 100pF 50V C0G
- D1, D2: value LTST-C190KGKT GREEN -> ASMT-RF45-AN002 YELLOW GREEN
- D1110: value LTST-C190KGKT -> ASMT-RF45-AN002 YELLOW GREEN
- D1111: value LTST-C190KFKT -> ASMT-RJ45-AQ502 ORANGE
- D1112: value LTST-C190KRKT -> ASMT-RR45-AQ902 RED
- D4: value BAT54H -> BAT54HT1G
- D900: footprint Diode_SMD:D_SOD-123F -> open-race-v2:SOD-123FL_Littelfuse_SMF
- F1: value 5A hold / 24V PTC -> 5.0A Ihold @23C / 24V PTC
- F900: value MF-PSMF010X (0.10A hold) -> MF-PSMF020X-2 (0.20A hold @23C)
- FB20, FB21: value 600R@100MHz 1A -> 600Ω @ 100MHz, 1.4A AEC-Q200; footprint Inductor_SMD:L_0805_2012Metric -> open-race-v2:FB_Murata_BLM21_2.0x1.25mm
- IC1: value AP33772SDKZ-13-FA01 -> AP33772SDKZ-13-FA02; footprint Package_DFN_QFN:WQFN-24-1EP_4x4mm_P0.5mm_EP2.45x2.45mm -> open-race-v2:WQFN-24-1EP_4x4mm_P0.5mm_EP2.70x2.70mm_AP33772S
- J800: value ESP UART PROGRAM (pin 1 VTREF only) -> M50-3530642 (VTREF sense only)
- J900: value U.FL / Beitian BT-T076 -> U.FL-R-SMT-1(10)
- L1: value 2.2uH XAL7030-222ME -> 2.2uH XAL7030-222MEC
- L20: value 1.5uH XFL4020-152ME -> 1.5uH XFL4020-152MEC
- L4: value 2.2nH -> 2.2nH 1A; footprint Inductor_SMD:L_1210_3225Metric -> open-race-v2:L_TDK_MHQ1005_1.0x0.6mm
- L8: value 18R @ 100MHz -> 22R @100MHz 8A; footprint Inductor_SMD:L_0603_1608Metric_Pad1.05x0.95mm_HandSolder -> Inductor_SMD:L_0603_1608Metric
- L900: value 68nH -> LQW18AN68NG00D 68nH 2%
- Q1, Q2, Q3, Q4, Q5: value NMOS -> CSD18540Q5B
- R11, R12: footprint Resistor_SMD:R_0603_1608Metric -> Resistor_SMD:R_1206_3216Metric
- R25: value 5.24k 1% -> 5.23k 1%
- R26: value 30.3k 1% -> 30.1k 1%
- SW1101: value BUTTON 1 -> KMR223NG ULC LFG
- SW1102: value BUTTON 2 -> KMR223NG ULC LFG
- SW1103: value BUTTON 3 -> KMR223NG ULC LFG
- SW300, SW801: value BOOT -> KMR223NG ULC LFG
- SW301: value DEV BOOT -> KMR223NG ULC LFG
- SW800: value RESET -> KMR223NG ULC LFG
- U10: footprint Package_DFN_QFN:Texas_RDX0007A_QFN-FCMOD-7-3.3x4mm-P0.5mm_4EP -> open-race-v2:Texas_RDX0007A_QFN-FCMOD-7-3.3x4mm-P0.5mm_4EP_NoVias
- U1000: value SCH16T-K01 -> SCH16T-K01-1
- U5: value MX25U51279GXDR00 -> IS25WP512M-RHLE
Connections:
- net /STM32 MCU I/O/BOOT0 renamed /STM32 MCU IO/BOOT0
- net /STM32 MCU I/O/DEV_BOOT renamed /STM32 MCU IO/DEV_BOOT
- net /STM32 MCU I/O/GNSS_ERR_STAT renamed /STM32 MCU IO/GNSS_ERR_STAT
- net /STM32 MCU I/O/GNSS_EVENT renamed /STM32 MCU IO/GNSS_EVENT
- net /STM32 MCU I/O/GNSS_PPS renamed /STM32 MCU IO/GNSS_PPS
- net /STM32 MCU I/O/GNSS_PVT_STAT renamed /STM32 MCU IO/GNSS_PVT_STAT
- net /STM32 MCU I/O/GNSS_RESET_N renamed /STM32 MCU IO/GNSS_RESET_N
- net /STM32 MCU I/O/GNSS_RTK_STAT renamed /STM32 MCU IO/GNSS_RTK_STAT
- net /STM32 MCU I/O/GNSS_UART_RX renamed /STM32 MCU IO/GNSS_UART_RX
- net /STM32 MCU I/O/GNSS_UART_TX renamed /STM32 MCU IO/GNSS_UART_TX
- net /STM32 MCU I/O/HSE_IN renamed /STM32 MCU IO/HSE_IN
- net /STM32 MCU I/O/HSE_OUT renamed /STM32 MCU IO/HSE_OUT
- net /STM32 MCU I/O/LSE_IN renamed /STM32 MCU IO/LSE_IN
- net /STM32 MCU I/O/LSE_OUT renamed /STM32 MCU IO/LSE_OUT
- net /STM32 MCU I/O/OTG1_TXRTUNE renamed /STM32 MCU IO/OTG1_TXRTUNE
- net /STM32 MCU I/O/PSRAM_CLK renamed /STM32 MCU IO/PSRAM_CLK
- net /STM32 MCU I/O/PSRAM_DQS0 renamed /STM32 MCU IO/PSRAM_DQS0
- net /STM32 MCU I/O/PSRAM_DQS1 renamed /STM32 MCU IO/PSRAM_DQS1
- net /STM32 MCU I/O/PSRAM_IO0 renamed /STM32 MCU IO/PSRAM_IO0
- net /STM32 MCU I/O/PSRAM_IO1 renamed /STM32 MCU IO/PSRAM_IO1
- net /STM32 MCU I/O/PSRAM_IO10 renamed /STM32 MCU IO/PSRAM_IO10
- net /STM32 MCU I/O/PSRAM_IO11 renamed /STM32 MCU IO/PSRAM_IO11
- net /STM32 MCU I/O/PSRAM_IO12 renamed /STM32 MCU IO/PSRAM_IO12
- net /STM32 MCU I/O/PSRAM_IO13 renamed /STM32 MCU IO/PSRAM_IO13
- net /STM32 MCU I/O/PSRAM_IO14 renamed /STM32 MCU IO/PSRAM_IO14
- net /STM32 MCU I/O/PSRAM_IO15 renamed /STM32 MCU IO/PSRAM_IO15
- net /STM32 MCU I/O/PSRAM_IO2 renamed /STM32 MCU IO/PSRAM_IO2
- net /STM32 MCU I/O/PSRAM_IO3 renamed /STM32 MCU IO/PSRAM_IO3
- net /STM32 MCU I/O/PSRAM_IO4 renamed /STM32 MCU IO/PSRAM_IO4
- net /STM32 MCU I/O/PSRAM_IO5 renamed /STM32 MCU IO/PSRAM_IO5
- net /STM32 MCU I/O/PSRAM_IO6 renamed /STM32 MCU IO/PSRAM_IO6
- net /STM32 MCU I/O/PSRAM_IO7 renamed /STM32 MCU IO/PSRAM_IO7
- net /STM32 MCU I/O/PSRAM_IO8 renamed /STM32 MCU IO/PSRAM_IO8
- net /STM32 MCU I/O/PSRAM_IO9 renamed /STM32 MCU IO/PSRAM_IO9
- net /STM32 MCU I/O/PSRAM_NCS renamed /STM32 MCU IO/PSRAM_NCS
- net /STM32 MCU I/O/SWCLK renamed /STM32 MCU IO/SWCLK
- net /STM32 MCU I/O/SWDIO renamed /STM32 MCU IO/SWDIO
- net /STM32 MCU I/O/SWO renamed /STM32 MCU IO/SWO
- net /STM32 MCU I/O/USBPD_INT renamed /STM32 MCU IO/USBPD_INT
- net /STM32 MCU I/O/USBPD_SCL renamed /STM32 MCU IO/USBPD_SCL
- net /STM32 MCU I/O/USBPD_SDA renamed /STM32 MCU IO/USBPD_SDA
- net /STM32 MCU I/O/USB_DN renamed /STM32 MCU IO/USB_DN
- net /STM32 MCU I/O/USB_DP renamed /STM32 MCU IO/USB_DP
- net /STM32 MCU I/O/USB_TPD8S_FLT renamed /STM32 MCU IO/USB_TPD8S_FLT
- net /STM32 MCU I/O/USB_VBUS_SENSE renamed /STM32 MCU IO/USB_VBUS_SENSE
- C304 pad 1: /STM32 MCU I/O/NRST -> NRST
- C6 pad 1: +3V3_MAIN -> /USB-C PD/USB_PROT_3V3_AON
- C901 pad 1: Net-(D900-A) -> Net-(D900-K)
- C902 pad 1: Net-(D900-A) -> Net-(D900-K)
- D4 pad 1: +1V8_RUN -> NRST
- D900 pad 1: GND -> Net-(D900-K)
- D900 pad 2: Net-(D900-A) -> GND
- F1 pad 1: /Power/PACK_POS -> /Power/PACK_POS_CONN
- F900 pad 2: Net-(D900-A) -> Net-(D900-K)
- J1 pad 3: /STM32 MCU I/O/NRST -> NRST
- J20 pad 1: /Power/PACK_POS -> /Power/PACK_POS_CONN
- J3 pad 1: /microSD/SD_D2 -> /STM32 MCU IO/SD_D2
- J3 pad 2: /microSD/SD_D3 -> /STM32 MCU IO/SD_D3
- J3 pad 3: /microSD/SD_CMD -> /STM32 MCU IO/SD_CMD
- J3 pad 5: /microSD/SD_CLK -> /STM32 MCU IO/SD_CLK
- J3 pad 7: /microSD/SD_D0 -> /STM32 MCU IO/SD_D0
- J3 pad 8: /microSD/SD_D1 -> /STM32 MCU IO/SD_D1
- J3 pad 9: /microSD/SD_CD_N -> /STM32 MCU IO/SD_CD_N
- L900 pad 2: Net-(D900-A) -> Net-(D900-K)
- Q1 pad 1: /USB-C PD/AP_VCC -> /USB-C PD/USB_PD_FET_COMMON
- Q1 pad 2: /USB-C PD/AP_VCC -> /USB-C PD/USB_PD_FET_COMMON
- Q1 pad 3: /USB-C PD/AP_VCC -> /USB-C PD/USB_PD_FET_COMMON
- Q1 pad 5: /USB-C PD/USB_PD_FET_COMMON -> /USB-C PD/AP_VCC
- Q1 pad 6: /USB-C PD/USB_PD_FET_COMMON -> /USB-C PD/AP_VCC
- Q1 pad 7: /USB-C PD/USB_PD_FET_COMMON -> /USB-C PD/AP_VCC
- Q1 pad 8: /USB-C PD/USB_PD_FET_COMMON -> /USB-C PD/AP_VCC
- Q2 pad 1: VBUS_PD -> /USB-C PD/USB_PD_FET_COMMON
- Q2 pad 2: VBUS_PD -> /USB-C PD/USB_PD_FET_COMMON
- Q2 pad 3: VBUS_PD -> /USB-C PD/USB_PD_FET_COMMON
- Q2 pad 5: /USB-C PD/USB_PD_FET_COMMON -> VBUS_PD
- Q2 pad 6: /USB-C PD/USB_PD_FET_COMMON -> VBUS_PD
- Q2 pad 7: /USB-C PD/USB_PD_FET_COMMON -> VBUS_PD
- Q2 pad 8: /USB-C PD/USB_PD_FET_COMMON -> VBUS_PD
- Q5 pad 1: Net-(Q5-S-Pad1) -> /Power/vpack+
- Q5 pad 2: Net-(Q5-S-Pad1) -> /Power/vpack+
- Q5 pad 3: Net-(Q5-S-Pad1) -> /Power/vpack+
- Q5 pad 4: unconnected-(Q5-G-Pad4) -> Net-(Q5-G)
- Q5 pad 5: Net-(Q5-D-Pad5) -> Net-(Q4-D-Pad5)
- Q5 pad 6: Net-(Q5-D-Pad5) -> Net-(Q4-D-Pad5)
- Q5 pad 7: Net-(Q5-D-Pad5) -> Net-(Q4-D-Pad5)
- Q5 pad 8: Net-(Q5-D-Pad5) -> Net-(Q4-D-Pad5)
- R14 pad 2: /microSD/SD_D0 -> /STM32 MCU IO/SD_D0
- R15 pad 2: /microSD/SD_D1 -> /STM32 MCU IO/SD_D1
- R16 pad 2: /microSD/SD_D2 -> /STM32 MCU IO/SD_D2
- R17 pad 2: /microSD/SD_D3 -> /STM32 MCU IO/SD_D3
- R18 pad 2: /microSD/SD_CMD -> /STM32 MCU IO/SD_CMD
- R19 pad 2: /microSD/SD_CD_N -> /STM32 MCU IO/SD_CD_N
- R300 pad 2: /STM32 MCU I/O/NRST -> NRST
- R8 pad 1: unconnected-(R8-Pad1) -> Net-(Q5-G)
- U1 pad A13: /STM32 MCU I/O/LED_RUN -> /Buttons and LEDs/LED_RUN
- U1 pad A8: /STM32 MCU I/O/SD_D2 -> /STM32 MCU IO/SD_D2
- U1 pad B1: /STM32 MCU I/O/SD_CD_N -> /STM32 MCU IO/SD_CD_N
- U1 pad B8: /STM32 MCU I/O/SD_D3 -> /STM32 MCU IO/SD_D3
- U1 pad C13: /STM32 MCU I/O/LED_ERR -> /Buttons and LEDs/LED_ERR
- U1 pad C7: /STM32 MCU I/O/SD_D1 -> /STM32 MCU IO/SD_D1
- U1 pad C8: /STM32 MCU I/O/SD_CLK -> /STM32 MCU IO/SD_CLK
- U1 pad D7: /STM32 MCU I/O/SD_D0 -> /STM32 MCU IO/SD_D0
- U1 pad E3: /STM32 MCU I/O/BTN3_N -> /Buttons and LEDs/BTN3_N
- U1 pad E4: /STM32 MCU I/O/BTN2_N -> /Buttons and LEDs/BTN2_N
- U1 pad E5: /STM32 MCU I/O/BTN1_N -> /Buttons and LEDs/BTN1_N
- U1 pad E7: /STM32 MCU I/O/SD_CMD -> /STM32 MCU IO/SD_CMD
- U1 pad G14: /STM32 MCU I/O/LED_WARN -> /Buttons and LEDs/LED_WARN
- U1 pad G3: /STM32 MCU I/O/NRST -> NRST
- U1 pad M3: unconnected-(U1B-PF5-PadM3) -> /ESP32-C6 radio/ESP_UART_RTS
- U1 pad T10: /ESP32-C6 radio/ESP_UART_RTS -> unconnected-(U1B-PG10-PadT10)
- U4 pad 10: +3V3_MAIN -> /USB-C PD/USB_PROT_3V3_AON
- U6 pad 24: Net-(Q3-G) -> Net-(U6-SDRV)

Commit message: pcb
Parts:
- moved U1 3.80 mm to (121.7, 98.3)
- moved U3 3.35 mm to (134.5, 94.0)
- moved U5 3.35 mm to (134.5, 101.5)
Connections:
- D4 pad 2: /Quad boot flash/FLASH_RESET_N -> unconnected-(D4-A-Pad2)
Routing:
- net Net-(C29-Pad1): track 0.00 -> 2.26 mm
- net unconnected-(U1B-PG5-PadM4): track 0.00 -> 0.57 mm
- net unconnected-(U1B-PF6-PadL5): track 0.00 -> 0.57 mm
- net unconnected-(U1B-PF10-PadL4): track 0.00 -> 0.57 mm
- net +1V8_RUN: track 0.00 -> 0.57 mm
- net unconnected-(U1B-PG6-PadL3): track 0.00 -> 0.57 mm
- net GND: track 0.00 -> 0.57 mm
- net /ESP32-C6 radio/ESP_UART_RTS: track 0.00 -> 0.57 mm
- net unconnected-(U1B-PF8-PadN3): track 0.00 -> 0.57 mm
- net unconnected-(U1A-PA11-PadT7): track 0.00 -> 0.57 mm
- net unconnected-(U1A-PA10-PadR7): track 0.00 -> 0.57 mm
- net /STM32 MCU IO/USB_VBUS_SENSE: track 0.00 -> 0.57 mm
- net unconnected-(U1B-PF4-PadL2): track 0.00 -> 0.57 mm
- net unconnected-(U1B-PF3-PadM2): track 0.00 -> 0.57 mm
- net unconnected-(U1B-PF14-PadN2): track 0.00 -> 0.57 mm
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
Commit message: pcb flash
Parts:
- D4: value BAT54HT1G -> BAT54XV2T1G; footprint Diode_SMD:D_SOD-323 -> Diode_SMD:D_SOD-523; moved to B.Cu
- R140, R303, R320, R321, R322, R323, R324, R325: moved to B.Cu
- moved R140 107.7 mm to (133.5, 103.5), turned to 90 degrees
- moved D4 106.7 mm to (131.7, 98.5)
- moved R303 102.6 mm to (133.0, 100.0), turned to 180 degrees
- moved R323 76.7 mm to (134.0, 102.0), turned to 180 degrees
- moved R321 76.4 mm to (130.9, 104.7), turned to 180 degrees
- moved R320 75.2 mm to (130.9, 103.7), turned to 180 degrees
- moved R322 73.7 mm to (130.9, 99.7), turned to 180 degrees
- moved R324 72.7 mm to (130.9, 100.7), turned to 180 degrees
- moved R325 72.4 mm to (130.9, 101.7), turned to 180 degrees
- moved U3 0.60 mm to (133.9, 94.2)
- moved U5 0.50 mm to (134.0, 101.5), turned to 90 degrees
- moved C80 0.09 mm to (85.0, 64.0)
Connections:
- D4 pad 2: unconnected-(D4-A-Pad2) -> /Quad boot flash/FLASH_RESET_N
Routing:
- net /Quad boot flash/FLASH_IO0: track 0.00 -> 8.66 mm, vias 0 -> 3
- net Net-(U1C-PN5): track 0.00 -> 6.97 mm, vias 0 -> 1
- net Net-(U1C-PN6): track 0.00 -> 4.88 mm, vias 0 -> 1
- net Net-(U1C-PN3): track 0.00 -> 4.66 mm, vias 0 -> 1
- net /Quad boot flash/FLASH_IO1: track 0.00 -> 4.50 mm, vias 0 -> 2
- net /Quad boot flash/FLASH_IO2: track 0.00 -> 4.10 mm, vias 0 -> 3
- net /Quad boot flash/FLASH_NCS: track 0.00 -> 3.34 mm, vias 0 -> 2
- net Net-(U1C-PN4): track 0.00 -> 3.04 mm, vias 0 -> 2
- net Net-(U1C-PN1): track 0.00 -> 2.85 mm, vias 0 -> 2
- net Net-(U1C-PN2): track 0.00 -> 2.69 mm, vias 0 -> 1
- net /Quad boot flash/FLASH_CLK: track 0.00 -> 2.46 mm, vias 0 -> 2
- net Net-(C29-Pad1): track 2.26 -> 0.00 mm
- net /Quad boot flash/FLASH_RESET_N: track 0.00 -> 2.21 mm, vias 0 -> 3
- net /Quad boot flash/FLASH_IO3: track 0.00 -> 1.71 mm, vias 0 -> 1
- net unconnected-(U1B-PG5-PadM4): track 0.57 -> 0.00 mm
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- added copper zone on In1.Cu, net GND

Commit message: remove resistors on flash line
Parts:
- removed R320, R321, R322, R323, R324, R325: 22R, Resistor_SMD:R_0402_1005Metric
- D4: moved to F.Cu
- moved D4 163.0 mm to (1.32, 0.72)
- moved R140 0.98 mm to (133.5, 102.5)
Connections:
- U1 pad G15: Net-(U1C-PP7) -> /STM32 MCU IO/PSRAM_IO7
- U1 pad G16: Net-(U1C-PP6) -> /STM32 MCU IO/PSRAM_IO6
- U1 pad G17: Net-(U1C-PP0) -> /STM32 MCU IO/PSRAM_IO0
- U1 pad H15: Net-(U1C-PP4) -> /STM32 MCU IO/PSRAM_IO4
- U1 pad H16: Net-(U1C-PP1) -> /STM32 MCU IO/PSRAM_IO1
- U1 pad H17: Net-(U1C-PP15) -> /STM32 MCU IO/PSRAM_IO15
- U1 pad J14: Net-(U1C-PP5) -> /STM32 MCU IO/PSRAM_IO5
- U1 pad J15: Net-(U1C-PP12) -> /STM32 MCU IO/PSRAM_IO12
- U1 pad J16: Net-(U1C-PP3) -> /STM32 MCU IO/PSRAM_IO3
- U1 pad J17: Net-(U1C-PP2) -> /STM32 MCU IO/PSRAM_IO2
- U1 pad K14: Net-(U1C-PP13) -> /STM32 MCU IO/PSRAM_IO13
- U1 pad K17: Net-(U1C-PO2) -> /STM32 MCU IO/PSRAM_DQS0
- U1 pad L15: Net-(U1C-PP11) -> /STM32 MCU IO/PSRAM_IO11
- U1 pad L16: Net-(U1C-PP8) -> /STM32 MCU IO/PSRAM_IO8
- U1 pad L17: Net-(U1C-PP14) -> /STM32 MCU IO/PSRAM_IO14
- U1 pad M16: Net-(U1C-PO3) -> /STM32 MCU IO/PSRAM_DQS1
- U1 pad M17: Net-(U1C-PO0) -> /STM32 MCU IO/PSRAM_NCS
- U1 pad N14: Net-(U1C-PP9) -> /STM32 MCU IO/PSRAM_IO9
- U1 pad N15: Net-(U1C-PP10) -> /STM32 MCU IO/PSRAM_IO10
- U1 pad N17: Net-(U1C-PN4) -> /Quad boot flash/FLASH_IO2
- U1 pad P15: Net-(U1C-PN6) -> /Quad boot flash/FLASH_CLK
- U1 pad R15: Net-(U1C-PN3) -> /Quad boot flash/FLASH_IO1
- U1 pad R16: Net-(U1C-PN5) -> /Quad boot flash/FLASH_IO3
- U1 pad R17: Net-(U1C-PN1) -> /Quad boot flash/FLASH_NCS
- U1 pad T17: Net-(U1C-PN2) -> /Quad boot flash/FLASH_IO0
Routing:
- net /Quad boot flash/FLASH_IO3: track 1.71 -> 9.54 mm, vias 1 -> 2
- net /Quad boot flash/FLASH_IO1: track 4.50 -> 11.6 mm
- net Net-(U1C-PN5): track 6.97 -> 0.00 mm, vias 1 -> 0
- net Net-(U1C-PN6): track 4.88 -> 0.00 mm, vias 1 -> 0
- net /Quad boot flash/FLASH_CLK: track 2.46 -> 7.16 mm
- net Net-(U1C-PN3): track 4.66 -> 0.00 mm, vias 1 -> 0
- net /Quad boot flash/FLASH_IO2: track 4.10 -> 8.16 mm, vias 3 -> 4
- net /Quad boot flash/FLASH_NCS: track 3.34 -> 6.56 mm, vias 2 -> 3
- net Net-(U1C-PN4): track 3.04 -> 0.00 mm, vias 2 -> 0
- net Net-(U1C-PN1): track 2.85 -> 0.00 mm, vias 2 -> 0
- net Net-(U1C-PN2): track 2.69 -> 0.00 mm, vias 1 -> 0
- net GND: track 0.71 -> 1.27 mm, vias 1 -> 2
- net /Quad boot flash/FLASH_IO0: track 8.66 -> 8.91 mm, vias 3 -> 2
- net /Quad boot flash/FLASH_RESET_N: vias 3 -> 2

Commit message: lsdfj" "s df l
Parts:
- removed R44, R45, R46, R47, R48, R49, R50, R51, R53, R54, R55, R56, R57, R59, R60, R61, R62, R63, R64: 22R, Resistor_SMD:R_0402_1005Metric
- D4, R174, R58: moved to B.Cu
- moved D4 163.1 mm to (131.7, 98.7)
- moved R58 82.0 mm to (135.9, 92.7)
- moved R174 79.5 mm to (135.9, 91.7)
- turned U3 to -90 degrees
Routing:
- net Net-(U1C-PO4): track 0.00 -> 15.0 mm, vias 0 -> 1
- net /STM32 MCU IO/PSRAM_IO14: track 0.00 -> 8.36 mm
- net /STM32 MCU IO/PSRAM_IO2: track 0.00 -> 8.29 mm
- net /STM32 MCU IO/PSRAM_IO15: track 0.00 -> 6.37 mm
- net /STM32 MCU IO/PSRAM_IO6: track 0.00 -> 6.08 mm
- net /STM32 MCU IO/PSRAM_IO0: track 0.00 -> 5.87 mm
- net /STM32 MCU IO/PSRAM_CLK: track 0.00 -> 1.70 mm, vias 0 -> 2
- net +1V8_RUN: track 0.72 -> 2.06 mm, vias 1 -> 3
- net GND: track 1.27 -> 2.48 mm, vias 2 -> 5
- net /STM32 MCU IO/PSRAM_NCS: track 0.00 -> 0.57 mm, vias 0 -> 1
- net /STM32 MCU IO/PSRAM_DQS1: track 0.00 -> 0.57 mm, vias 0 -> 1
- net /STM32 MCU IO/PSRAM_IO9: track 0.00 -> 0.57 mm, vias 0 -> 1
- net /STM32 MCU IO/PSRAM_IO13: track 0.00 -> 0.57 mm
- net /STM32 MCU IO/PSRAM_IO10: track 0.00 -> 0.57 mm, vias 0 -> 1
- net /STM32 MCU IO/USB_TPD8S_FLT: track 0.00 -> 0.57 mm, vias 0 -> 1
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
Commit message: finish ram fanout
Parts:
- moved C142 30.8 mm to (98.0, 51.4)
- moved C141 27.3 mm to (95.4, 46.7)
- moved C144 27.3 mm to (91.9, 45.5)
- moved C143 27.3 mm to (91.9, 43.0)
- moved R302 21.8 mm to (95.4, 44.7)
- moved D4 2.19 mm to (130.6, 100.6)
Routing:
- net /STM32 MCU IO/PSRAM_IO9: track 0.57 -> 17.5 mm, vias 1 -> 2
- net /STM32 MCU IO/PSRAM_IO10: track 0.57 -> 15.6 mm, vias 1 -> 2
- net /STM32 MCU IO/PSRAM_IO8: track 0.00 -> 15.0 mm, vias 0 -> 2
- net /STM32 MCU IO/PSRAM_IO12: track 0.00 -> 13.6 mm, vias 0 -> 2
- net /STM32 MCU IO/PSRAM_DQS1: track 0.57 -> 13.8 mm, vias 1 -> 0
- net /STM32 MCU IO/PSRAM_NCS: track 0.57 -> 13.6 mm, vias 1 -> 0
- net /STM32 MCU IO/PSRAM_IO3: track 0.00 -> 12.4 mm, vias 0 -> 2
- net /STM32 MCU IO/PSRAM_IO11: track 0.00 -> 11.4 mm, vias 0 -> 2
- net /STM32 MCU IO/PSRAM_IO13: track 0.57 -> 11.2 mm, vias 0 -> 2
- net /STM32 MCU IO/PSRAM_DQS0: track 0.00 -> 8.66 mm, vias 0 -> 2
- net /STM32 MCU IO/PSRAM_IO5: track 0.00 -> 7.93 mm, vias 0 -> 2
- net /STM32 MCU IO/PSRAM_IO1: track 0.00 -> 7.66 mm, vias 0 -> 2
- net /STM32 MCU IO/PSRAM_IO4: track 0.00 -> 7.30 mm, vias 0 -> 2
- net /STM32 MCU IO/PSRAM_IO7: track 0.00 -> 7.30 mm, vias 0 -> 2
- net +1V8_RUN: track 2.06 -> 5.68 mm, vias 3 -> 4
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
Commit message: lengthmatch
Routing:
- net /STM32 MCU IO/PSRAM_IO15: track 6.38 -> 9.75 mm
- net /STM32 MCU IO/PSRAM_IO14: track 8.36 -> 10.0 mm
- net /STM32 MCU IO/PSRAM_NCS: track 13.6 -> 12.7 mm
