File: pcb/v2_mini_pcb/IMU_Mini.kicad_sch (KiCad schematic)
At the start: 7 parts, among them U7 SCH16T-K01

Commit message: finish v2_mini schematic
Changed lines of the file:
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@@
+	)
+	(junction
+		(at 114.3 77.47)
+		(diameter 0)
+		(color 0 0 0 0)
 	)
 	(junction
@@
 	)
 	(junction
+		(at 137.16 85.09)
+		(diameter 0)
+		(color 0 0 0 0)
+	)
+	(junction
 		(at 113.03 125.73)
 		(diameter 0)
@@
 	)
 	(junction
-		(at 114.3 77.47)
-		(diameter 0)
-		(color 0 0 0 0)
-	)
-	(junction
 		(at 124.46 87.63)
-		(diameter 0)
-		(color 0 0 0 0)
-	)
-	(junction
-		(at 137.16 85.09)
 		(diameter 0)
 		(color 0 0 0 0)
@@
 	(wire
 		(pts
+			(xy 114.3 76.2) (xy 114.3 77.47)
+		)
+		(stroke
+			(width 0)
+			(type default)
+		)
+	)
+	(wire
+		(pts
 			(xy 135.89 38.1) (xy 156.21 38.1)
 		)
@@
 		(pts
 			(xy 113.03 90.17) (xy 133.35 90.17)
+		)
+		(stroke
+			(width 0)
+			(type default)
+		)
+	)
+	(wire
+		(pts
+			(xy 138.43 85.09) (xy 137.16 85.09)
 		)
 		(stroke
@@
 	(symbol
 		(lib_id "power:GND")
-		(at 114.3 77.47 180)
+		(at 114.3 76.2 180)
 		(unit 1)
 		(body_style 1)
@@
 		(fields_autoplaced yes)
 		(property "Reference" "#PWR07"
+			(at 114.3 69.85 0)
+			(hide yes)
+			(show_name no)
+			(do_not_autoplace no)
+			(effects
+				(font
+					(size 1.27 1.27)
+				)
+			)
+		)
+		(property "Value" "GND"
 			(at 114.3 71.12 0)
-			(hide yes)
-			(show_name no)
-			(do_not_autoplace no)
-			(effects
-				(font
-					(size 1.27 1.27)
-				)
-			)
-		)
-		(property "Value" "GND"
-			(at 114.3 72.39 0)
 			(show_name no)
 			(do_not_autoplace no)
@@
 		)
 		(property "Footprint" ""
-			(at 114.3 77.47 0)
+			(at 114.3 76.2 0)
 			(hide yes)
 			(show_name no)
@@
 		)
 		(property "Datasheet" ""
-			(at 114.3 77.47 0)
+			(at 114.3 76.2 0)
 			(hide yes)
 			(show_name no)
@@
 		)
 		(property "Description" "Power symbol creates a global label with name \"GND\" , ground"
-			(at 114.3 77.47 0)
+			(at 114.3 76.2 0)
 			(hide yes)
 			(show_name no)
@@
 	(symbol
 		(lib_id "power:PWR_FLAG")
-		(at 137.16 85.09 270)
+		(at 138.43 85.09 270)
 		(unit 1)
 		(body_style 1)
@@
 		(fields_autoplaced yes)
 		(property "Reference" "#FLG06"
-			(at 139.065 85.09 0)
+			(at 140.335 85.09 0)
 			(hide yes)
 			(show_name no)
@@
 		)
 		(property "Value" "+3V3_IMU"
-			(at 140.97 85.0899 90)
+			(at 142.24 85.0899 90)
 			(show_name no)
 			(do_not_autoplace no)
@@
 		)
 		(property "Footprint" ""
-			(at 137.16 85.09 0)
+			(at 138.43 85.09 0)
 			(hide yes)
 			(show_name no)
@@
 		)
 		(property "Datasheet" ""
-			(at 137.16 85.09 0)
+			(at 138.43 85.09 0)
 			(hide yes)
 			(show_name no)
@@
 		)
 		(property "Description" "Special symbol for telling ERC where power comes from"
-			(at 137.16 85.09 0)
-			(hide yes)
-			(show_name no)
+			(at 138.43 85.09 0)
+			(hide yes)
+			(show_name no)

Commit message: fix minor edc rules
Parts:
- removed C25: 10uF, symbol Device:C_Small
- removed C26, C28: 1uF, symbol Device:C_Small
- removed C27, C29: 100nF, symbol Device:C_Small
- removed R20: 10k, symbol Device:R_Small_US
- removed U7: SCH16T-K01, SCH16T-K10-10:XDCR_SCH16T-K10-10, symbol all:SCH16T-K10-10
- added C36: 10uF, symbol Device:C_Small
- added C37, C39: 1uF, symbol Device:C_Small
- added C38, C40: 100nF, symbol Device:C_Small
- added R27: 10k, symbol Device:R_Small_US
- added U3: SCH16T-K01-1, SCH16T-K01-1:XDCR_SCH16T-K01-1, symbol all:SCH16T-K01-1
Connections:
- net GND: now also C36.2, C37.2, C38.1, C39.1, C40.1, U3.1 (HEATSINK), U3.12 (GND), U3.13 (GND), U3.16 (GND), U3.2 (RESERVED), U3.24 (HEATSINK), U3.3 (TA9), U3.4 (TA8), U3.5 (RESERVED), U3.7 (RESERVED), U3.9 (GND)
- net IMU_CS_N: now also U3.22 (CS)
- net IMU_DRDY: now also U3.20 (DRY_SYNC)
- net IMU_MISO: now also U3.19 (MISO)
- net IMU_MOSI: now also U3.23 (MOSI)
- net IMU_RESET_N: now also R27.2, U3.6 (~{EXTRES})
- net IMU_SCLK: now also U3.21 (SCK)
- new net: C36.1, U3.10 (VREGA2), U3.11 (VREGA)
- new net: C37.1, U3.14 (VREGD2), U3.15 (VREGD)
- new net V3P3: C38.2, C39.2, C40.2, U3.17 (V3P3), U3.18 (VDDIO), U3.8 (V3P3)
- no-connect marks 1 -> 0
Other:
- note removed: "Place U6 on the rigid mounting region. Record sensor axes on copper/silkscreen; keep switching stages, connectors and button forces away."

Commit message: erc rules
Parts:
- removed R27: 10k, symbol Device:R_Small_US
- added R20: 10k, symbol Device:R_Small_US
Connections:
- net IMU_RESET_N: now also R20.2
- net V3P3: now also R20.1
Changed lines of the file:
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@@
 	(paper "A4")
+	(junction
+		(at 87.63 53.34)
+		(diameter 0)
+		(color 0 0 0 0)
+	)
 	(junction
 		(at 87.63 88.9)
@@
 	)
 	(junction
-		(at 38.1 68.58)
+		(at 87.63 71.12)
 		(diameter 0)
 		(color 0 0 0 0)
 	)
 	(junction
-		(at 87.63 71.12)
+		(at 36.83 68.58)
 		(diameter 0)
 		(color 0 0 0 0)
@@
 	(wire
 		(pts
+			(xy 36.83 40.64) (xy 36.83 62.23)
+		)
+		(stroke
+			(width 0)
+			(type default)
+		)
+	)
+	(wire
+		(pts
 			(xy 99.06 46.99) (xy 107.95 46.99)
 		)
@@
 	(wire
 		(pts
-			(xy 33.02 68.58) (xy 38.1 68.58)
-		)
-		(stroke
-			(width 0)
-			(type default)
-		)
-	)
-	(wire
-		(pts
 			(xy 88.9 45.72) (xy 88.9 46.99)
 		)
@@
 		)
 	)
-	(wire
-		(pts
-			(xy 38.1 67.31) (xy 38.1 68.58)
-		)
-		(stroke
-			(width 0)
-			(type default)
-		)
-	)
 	(bus
 		(pts
@@
 	(wire
 		(pts
-			(xy 38.1 60.96) (xy 38.1 62.23)
+			(xy 36.83 67.31) (xy 36.83 68.58)
 		)
 		(stroke
@@
 	(wire
 		(pts
+			(xy 36.83 68.58) (xy 46.99 68.58)
+		)
+		(stroke
+			(width 0)
+			(type default)
+		)
+	)
+	(wire
+		(pts
+			(xy 36.83 40.64) (xy 87.63 40.64)
+		)
+		(stroke
+			(width 0)
+			(type default)
+		)
+	)
+	(wire
+		(pts
 			(xy 87.63 60.96) (xy 87.63 63.5)
 		)
@@
 	(wire
 		(pts
+			(xy 87.63 40.64) (xy 87.63 53.34)
+		)
+		(stroke
+			(width 0)
+			(type default)
+		)
+	)
+	(wire
+		(pts
 			(xy 135.89 58.42) (xy 156.21 58.42)
 		)
@@
 	(wire
 		(pts
-			(xy 38.1 68.58) (xy 46.99 68.58)
-		)
-		(stroke
-			(width 0)
-			(type default)
-		)
-	)
-	(wire
-		(pts
 			(xy 135.89 43.18) (xy 156.21 43.18)
 		)
@@
 		(pts
 			(xy 87.63 81.28) (xy 107.95 81.28)
+		)
+		(stroke
+			(width 0)
+			(type default)
+		)
+	)
+	(wire
+		(pts
+			(xy 33.02 68.58) (xy 36.83 68.58)
 		)
 		(stroke
@@
 	)
 	(symbol
-		(lib_id "Device:R_Small_US")
-		(at 38.1 64.77 0)
-		(unit 1)
-		(body_style 1)
-		(exclude_from_sim no)
-		(in_bom yes)
-		(on_board yes)
-		(in_pos_files yes)
-		(dnp no)
-		(fields_autoplaced yes)
-		(property "Reference" "R27"
-			(at 40.64 63.4999 0)
-			(show_name no)
-			(do_not_autoplace no)
-			(effects
-				(font
-					(size 1.27 1.27)
-				)
-				(justify left)
-			)
-		)
-		(property "Value" "10k"
-			(at 40.64 66.0399 0)
-			(show_name no)
-			(do_not_autoplace no)
-			(effects
-				(font
-					(size 1.27 1.27)
-				)
-				(justify left)
-			)
-		)
-		(property "Footprint" ""
-			(at 38.1 64.77 0)
-			(hide yes)
-			(show_name no)
-			(do_not_autoplace no)
-			(effects
-				(font
-					(size 1.27 1.27)
-				)
-			)
-		)
-		(property "Datasheet" ""
-			(at 38.1 64.77 0)
-			(hide yes)
-			(show_name no)
-			(do_not_autoplace no)
-			(effects
-				(font
-					(size 1.27 1.27)
-				)
-			)
-		)
-		(property "Description" "Resistor, small US symbol"
-			(at 38.1 64.77 0)
-			(hide yes)
-			(show_name no)
-			(do_not_autoplace no)
-			(effects
-				(font
-					(size 1.27 1.27)
-				)
-			)
-		)
-		(pin "1"
-		)
-		(pin "2"
-		)
-		(instances
-			(project "v2_mini"
-				(path "/4318b369-034c-40ef-a05b-b7d2541c0647/a7e9176c-19e9-4164-84c0-42ef6ac15138"
-					(reference "R27")
-					(unit 1)
-				)
-			)
-		)
-	)
-	(symbol
 		(lib_id "Device:C_Small")
 		(at 99.06 49.53 0)
@@
 	)
 	(symbol
-		(lib_id "power:PWR_FLAG")
-		(at 38.1 60.96 0)
+		(lib_id "Device:R_Small_US")
+		(at 36.83 64.77 0)
 		(unit 1)
 		(body_style 1)
@@
 		(dnp no)
 		(fields_autoplaced yes)
-		(property "Reference" "#FLG011"
-			(at 38.1 59.055 0)
-			(hide yes)
-			(show_name no)
-			(do_not_autoplace no)
-			(effects
-				(font
-					(size 1.27 1.27)
-				)
-			)
-		)
-		(property "Value" "+3V3_IMU"
-			(at 38.1 55.88 0)
-			(show_name no)
-			(do_not_autoplace no)
-			(effects
-				(font
-					(size 1.27 1.27)
-				)
+		(property "Reference" "R20"
+			(at 39.37 63.4999 0)
+			(show_name no)
+			(do_not_autoplace no)
+			(effects
+				(font
+					(size 1.27 1.27)
+				)
+				(justify left)
+			)
+		)
+		(property "Value" "10k"
+			(at 39.37 66.0399 0)
+			(show_name no)
+			(do_not_autoplace no)
+			(effects
+				(font
+					(size 1.27 1.27)
+				)
+				(justify left)
 			)
 		)
 		(property "Footprint" ""
-			(at 38.1 60.96 0)
+			(at 36.83 64.77 0)
 			(hide yes)
 			(show_name no)
@@
 		)
 		(property "Datasheet" ""
-			(at 38.1 60.96 0)
-			(hide yes)
-			(show_name no)
-			(do_not_autoplace no)
-			(effects
-				(font
-					(size 1.27 1.27)
-				)
-			)
-		)
-		(property "Description" "Special symbol for telling ERC where power comes from"
-			(at 38.1 60.96 0)
+			(at 36.83 64.77 0)
+			(hide yes)
+			(show_name no)
+			(do_not_autoplace no)
+			(effects
+				(font
+					(size 1.27 1.27)
+				)
+			)
+		)
+		(property "Description" "Resistor, small US symbol"
+			(at 36.83 64.77 0)
 			(hide yes)
 			(show_name no)
@@
 		)
 		(pin "1"
+		)
+		(pin "2"
 		)
 		(instances
 			(project "v2_mini"
 				(path "/4318b369-034c-40ef-a05b-b7d2541c0647/a7e9176c-19e9-4164-84c0-42ef6ac15138"
-					(reference "#FLG011")
+					(reference "R20")
 					(unit 1)
 				)
