File: pcb/v2_mini_pcb/Power_USB.kicad_sch (KiCad schematic)
At the start: 32 parts, among them J6 USB4105-GF-A, U10 TPS63802DLAR, U6 TPD4EUSB30, U8 BQ25622RYKR, U9 MAX17048G_T10

Commit message: power done
Parts:
- added FB1, FB2: BLM21SP601SN1D, symbol Device:FerriteBead_Small
Connections:
- net +3V3: now also FB1.1, FB2.1
Changed lines of the file:
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@@
 	(wire
 		(pts
+			(xy 123.19 166.37) (xy 114.3 166.37)
+		)
+		(stroke
+			(width 0)
+			(type default)
+		)
+	)
+	(wire
+		(pts
 			(xy 205.74 104.14) (xy 213.36 104.14)
 		)
@@
 	(wire
 		(pts
+			(xy 121.92 157.48) (xy 114.3 157.48)
+		)
+		(stroke
+			(width 0)
+			(type default)
+		)
+	)
+	(wire
+		(pts
 			(xy 143.51 124.46) (xy 153.67 124.46)
 		)
@@
 	(wire
 		(pts
-			(xy 100.33 157.48) (xy 106.68 157.48)
+			(xy 100.33 157.48) (xy 109.22 157.48)
 		)
 		(stroke
@@
 	(wire
 		(pts
-			(xy 100.33 166.37) (xy 106.68 166.37)
+			(xy 100.33 166.37) (xy 109.22 166.37)
 		)
 		(stroke
@@
 	(symbol
 		(lib_id "power:PWR_FLAG")
-		(at 106.68 166.37 270)
+		(at 123.19 166.37 270)
 		(unit 1)
 		(body_style 1)
@@
 		(fields_autoplaced yes)
 		(property "Reference" "#FLG08"
-			(at 108.585 166.37 0)
+			(at 125.095 166.37 0)
 			(hide yes)
 			(show_name no)
@@
 		)
 		(property "Value" "+3V3_IMU"
-			(at 110.49 166.3699 90)
+			(at 127 166.3699 90)
 			(show_name no)
 			(do_not_autoplace no)
@@
 		)
 		(property "Footprint" ""
-			(at 106.68 166.37 0)
+			(at 123.19 166.37 0)
 			(hide yes)
 			(show_name no)
@@
 		)
 		(property "Datasheet" ""
-			(at 106.68 166.37 0)
+			(at 123.19 166.37 0)
 			(hide yes)
 			(show_name no)
@@
 		)
 		(property "Description" "Special symbol for telling ERC where power comes from"
-			(at 106.68 166.37 0)
+			(at 123.19 166.37 0)
 			(hide yes)
 			(show_name no)
@@
 	)
 	(symbol
+		(lib_id "Device:FerriteBead_Small")
+		(at 111.76 166.37 90)
+		(unit 1)
+		(body_style 1)
+		(exclude_from_sim no)
+		(in_bom yes)
+		(on_board yes)
+		(in_pos_files yes)
+		(dnp no)
+		(fields_autoplaced yes)
+		(property "Reference" "FB2"
+			(at 111.7219 160.02 90)
+			(show_name no)
+			(do_not_autoplace no)
+			(effects
+				(font
+					(size 1.27 1.27)
+				)
+			)
+		)
+		(property "Value" "BLM21SP601SN1D"
+			(at 111.7219 162.56 90)
+			(show_name no)
+			(do_not_autoplace no)
+			(effects
+				(font
+					(size 1.27 1.27)
+				)
+			)
+		)
+		(property "Footprint" ""
+			(at 111.76 168.148 90)
+			(hide yes)
+			(show_name no)
+			(do_not_autoplace no)
+			(effects
+				(font
+					(size 1.27 1.27)
+				)
+			)
+		)
+		(property "Datasheet" ""
+			(at 111.76 166.37 0)
+			(hide yes)
+			(show_name no)
+			(do_not_autoplace no)
+			(effects
+				(font
+					(size 1.27 1.27)
+				)
+			)
+		)
+		(property "Description" "Ferrite bead, small symbol"
+			(at 111.76 166.37 0)
+			(hide yes)
+			(show_name no)
+			(do_not_autoplace no)
+			(effects
+				(font
+					(size 1.27 1.27)
+				)
+			)
+		)
+		(pin "1"
+		)
+		(pin "2"
+		)
+		(instances
+			(project "v2_mini"
+				(path "/4318b369-034c-40ef-a05b-b7d2541c0647/4f258941-373d-43ad-86e2-121941fb93df"
+					(reference "FB2")
+					(unit 1)
+				)
+			)
+		)
+	)
+	(symbol
 		(lib_id "power:PWR_FLAG")
-		(at 106.68 157.48 270)
+		(at 121.92 157.48 270)
 		(unit 1)
 		(body_style 1)
@@
 		(fields_autoplaced yes)
 		(property "Reference" "#FLG01"
-			(at 108.585 157.48 0)
+			(at 123.825 157.48 0)
 			(hide yes)
 			(show_name no)
@@
 		)
 		(property "Value" "+3V3_GNSS"
-			(at 110.49 157.4799 90)
+			(at 125.73 157.4799 90)
 			(show_name no)
 			(do_not_autoplace no)
@@
 		)
 		(property "Footprint" ""
-			(at 106.68 157.48 0)
+			(at 121.92 157.48 0)
 			(hide yes)
 			(show_name no)
@@
 		)
 		(property "Datasheet" ""
-			(at 106.68 157.48 0)
+			(at 121.92 157.48 0)
 			(hide yes)
 			(show_name no)
@@
 		)
 		(property "Description" "Special symbol for telling ERC where power comes from"
-			(at 106.68 157.48 0)
+			(at 121.92 157.48 0)
 			(hide yes)
 			(show_name no)
@@
 					(unit 1)
 				)
+			)
+		)
+	)
+	(symbol
+		(lib_id "Device:FerriteBead_Small")
+		(at 111.76 157.48 90)
+		(unit 1)
+		(body_style 1)
+		(exclude_from_sim no)
+		(in_bom yes)
+		(on_board yes)
+		(in_pos_files yes)
+		(dnp no)
+		(fields_autoplaced yes)
+		(property "Reference" "FB1"
+			(at 111.7219 151.13 90)
+			(show_name no)
+			(do_not_autoplace no)
+			(effects
+				(font
+					(size 1.27 1.27)
+				)
+			)
+		)
+		(property "Value" "BLM21SP601SN1D"
+			(at 111.7219 153.67 90)
+			(show_name no)
+			(do_not_autoplace no)
+			(effects
+				(font
+					(size 1.27 1.27)
+				)
+			)
+		)
+		(property "Footprint" ""
+			(at 111.76 159.258 90)
+			(hide yes)
+			(show_name no)
+			(do_not_autoplace no)
+			(effects
+				(font
+					(size 1.27 1.27)
+				)
+			)
+		)
+		(property "Datasheet" ""
+			(at 111.76 157.48 0)
+			(hide yes)
+			(show_name no)
+			(do_not_autoplace no)
+			(effects
+				(font
+					(size 1.27 1.27)
+				)
+			)
+		)
+		(property "Description" "Ferrite bead, small symbol"
+			(at 111.76 157.48 0)
+			(hide yes)
+			(show_name no)
+			(do_not_autoplace no)
+			(effects
+				(font
+					(size 1.27 1.27)
+				)
+			)
+		)
+		(pin "1"
+		)
+		(pin "2"
+		)
+		(instances
+			(project "v2_mini"
+				(path "/4318b369-034c-40ef-a05b-b7d2541c0647/4f258941-373d-43ad-86e2-121941fb93df"
+					(reference "FB1")
+					(unit 1)
+				)

Commit message: fix minor edc rules
Connections:
- net BAT_SCL: now also U9.7 (SCL); no longer U9.8 (SDA)
- net BAT_SDA: now also U9.8 (SDA); no longer U9.7 (SCL)
- net +3V3_IMU: now reaches FB2.2
- net +3V3_GNSS: now reaches FB1.2

Commit message: erc rules
Parts:
- removed R24: 10k, symbol Device:R_Small_US
- added R3: 10k, symbol Device:R_Small_US
Connections:
- net +3V3: now also R3.1
- net BAT_ALRT: now also R3.2
- net BAT_SCL renamed POW_SCL
- net BAT_SDA renamed POW_SDA
Other:
- moved on the sheet: R16, R21
