File: pcb/v2_mini_pcb/Power_USB.kicad_sch (KiCad schematic)
At the start: 44 parts, among them J4 Battery, J6 USB4105-GF-A, SW7 SW_Push, U10 TPS63802DLAR, U6 TPD4EUSB30, U7 MAX16169AALTA+T, U8 BQ25622ERYKR, U9 MAX17048G_T10

Commit message: minor changes
Parts:
- J4: MPN (none) -> DF58-2P-1.2V(21)
