File: pcb/v2_mini_pcb/v2_mini.kicad_sch (KiCad schematic)
At the start: 0 parts

Commit message: fix minor edc rules
Other:
- sheet ESP32-S31 MCU ports: added {LCD}, {POWER_I2C}, {SD}; removed {CHARGER_I2C}, {HMI_IF}, {SHARED_SPI}
- sheet Power + USB ports: added {POWER_I2C}; removed {CHARGER_I2C}
- sheet Storage + Display ports: added {LCD}, {SD}; removed {HMI_IF}, {SHARED_SPI}

Commit message: finish footprint matching
Other:
- added sheet HID (hid.kicad_sch)
- sheet ESP32-S31 MCU ports: added {HID}; removed none
Changed lines of the file:
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@@
+	(bus
+		(pts
+			(xy 140.97 115.57) (xy 140.97 127)
+		)
+		(stroke
+			(width 0)
+			(type default)
+		)
+	)
 	(bus
 		(pts
@@
 	)
 	(sheet
+		(at 127 127)
+		(size 26.67 15.24)
+		(exclude_from_sim no)
+		(in_bom yes)
+		(on_board yes)
+		(dnp no)
+		(fields_autoplaced yes)
+		(stroke
+			(width 0.1524)
+			(type solid)
+		)
+		(fill
+			(color 0 0 0 0)
+		)
+		(property "Sheetname" "HID"
+			(at 127 126.2884 0)
+			(show_name no)
+			(do_not_autoplace no)
+			(effects
+				(font
+					(size 1.27 1.27)
+				)
+				(justify left bottom)
+			)
+		)
+		(property "Sheetfile" "hid.kicad_sch"
+			(at 127 142.8246 0)
+			(show_name no)
+			(do_not_autoplace no)
+			(effects
+				(font
+					(size 1.27 1.27)
+				)
+				(justify left top)
+			)
+		)
+		(pin "{HID}" bidirectional
+			(at 140.97 127 90)
+			(effects
+				(font
+					(size 1.27 1.27)
+				)
+				(justify right)
+			)
+		)
+		(instances
+			(project "v2_mini"
+				(path "/4318b369-034c-40ef-a05b-b7d2541c0647"
+					(page "7")
+				)
+			)
+		)
+	)
+	(sheet
 		(at 177.8 50.07)
 		(size 39.37 26.13)
@@
 			(effects
 				(font
+					(size 1.27 1.27)
+				)
+				(justify left)
+			)
+		)
+		(pin "{HID}" bidirectional
+			(at 140.97 115.57 270)
+			(effects
+				(font
