File: pcb/v2_mini_pcb/MCU.kicad_sch (KiCad schematic)
At the start: 20 parts, among them J5 TC2030, SW1 SW_Push, SW2 SW_Push

Commit message: add input buttons
Changed lines of the file:
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@@
 	)
 	(bus_entry
-		(at 212.09 46.99)
+		(at 207.01 46.99)
 		(size -2.54 2.54)
 		(stroke
@@
 	)
 	(bus_entry
-		(at 212.09 41.91)
+		(at 207.01 41.91)
 		(size -2.54 2.54)
 		(stroke
@@
 	)
 	(bus_entry
-		(at 254 44.45)
+		(at 232.41 41.91)
 		(size -2.54 2.54)
 		(stroke
@@
 	)
 	(bus_entry
-		(at 254 34.29)
+		(at 232.41 31.75)
 		(size -2.54 2.54)
 		(stroke
@@
 	)
 	(bus_entry
-		(at 254 39.37)
+		(at 232.41 36.83)
 		(size -2.54 2.54)
 		(stroke
@@
 	)
 	(bus_entry
-		(at 212.09 36.83)
+		(at 207.01 36.83)
 		(size -2.54 2.54)
 		(stroke
@@
 	)
 	(bus_entry
-		(at 212.09 31.75)
+		(at 207.01 31.75)
 		(size -2.54 2.54)
 		(stroke
@@
 	)
 	(bus_entry
-		(at 212.09 52.07)
+		(at 207.01 52.07)
 		(size -2.54 2.54)
 		(stroke
@@
 	)
 	(bus_entry
-		(at 212.09 57.15)
+		(at 207.01 57.15)
 		(size -2.54 2.54)
 		(stroke
@@
 	)
 	(bus_entry
-		(at 212.09 62.23)
+		(at 207.01 62.23)
 		(size -2.54 2.54)
 		(stroke
@@
 	(wire
 		(pts
-			(xy 209.55 44.45) (xy 194.31 44.45)
+			(xy 204.47 44.45) (xy 189.23 44.45)
 		)
 		(stroke
@@
 	(wire
 		(pts
-			(xy 209.55 39.37) (xy 194.31 39.37)
+			(xy 204.47 39.37) (xy 189.23 39.37)
 		)
 		(stroke
@@
 	(wire
 		(pts
-			(xy 209.55 64.77) (xy 194.31 64.77)
+			(xy 204.47 64.77) (xy 189.23 64.77)
 		)
 		(stroke
@@
 	(bus
 		(pts
-			(xy 212.09 46.99) (xy 212.09 52.07)
+			(xy 207.01 46.99) (xy 207.01 52.07)
 		)
 		(stroke
@@
 	(bus
 		(pts
-			(xy 212.09 52.07) (xy 212.09 57.15)
+			(xy 207.01 52.07) (xy 207.01 57.15)
 		)
 		(stroke
@@
 	(wire
 		(pts
-			(xy 236.22 36.83) (xy 251.46 36.83)
+			(xy 214.63 34.29) (xy 229.87 34.29)
 		)
 		(stroke
@@
 	(wire
 		(pts
-			(xy 251.46 41.91) (xy 236.22 41.91)
+			(xy 229.87 39.37) (xy 214.63 39.37)
 		)
 		(stroke
@@
 	(bus
 		(pts
-			(xy 212.09 57.15) (xy 212.09 62.23)
+			(xy 207.01 57.15) (xy 207.01 62.23)
 		)
 		(stroke
@@
 	(bus
 		(pts
-			(xy 212.09 26.67) (xy 212.09 46.99)
+			(xy 207.01 26.67) (xy 207.01 46.99)
 		)
 		(stroke
@@
 	(wire
 		(pts
-			(xy 194.31 34.29) (xy 209.55 34.29)
+			(xy 189.23 34.29) (xy 204.47 34.29)
 		)
 		(stroke
@@
 	(wire
 		(pts
-			(xy 209.55 54.61) (xy 194.31 54.61)
+			(xy 204.47 54.61) (xy 189.23 54.61)
 		)
 		(stroke
@@
 	(bus
 		(pts
-			(xy 254 29.21) (xy 254 44.45)
+			(xy 232.41 26.67) (xy 232.41 41.91)
 		)
 		(stroke
@@
 	(wire
 		(pts
-			(xy 209.55 59.69) (xy 194.31 59.69)
+			(xy 204.47 59.69) (xy 189.23 59.69)
 		)
 		(stroke
@@
 	(wire
 		(pts
-			(xy 209.55 49.53) (xy 194.31 49.53)
+			(xy 204.47 49.53) (xy 189.23 49.53)
 		)
 		(stroke
@@
 	(wire
 		(pts
-			(xy 251.46 46.99) (xy 236.22 46.99)
+			(xy 229.87 44.45) (xy 214.63 44.45)
 		)
 		(stroke
@@
 	)
 	(label "LCD_DC"
-		(at 194.31 54.61 0)
+		(at 189.23 54.61 0)
 		(effects
 			(font
@@
 	)
 	(label "HDI_SCL"
-		(at 236.22 36.83 0)
+		(at 214.63 34.29 0)
 		(effects
 			(font
@@
 	)
 	(label "LCD_TE"
-		(at 194.31 64.77 0)
+		(at 189.23 64.77 0)
 		(effects
 			(font
@@
 	)
 	(label "LCD_CSN"
-		(at 194.31 44.45 0)
+		(at 189.23 44.45 0)
 		(effects
 			(font
@@
 	)
 	(label "LCD_RN"
-		(at 194.31 34.29 0)
+		(at 189.23 34.29 0)
 		(effects
 			(font
@@
 	)
 	(label "LCD_SDA"
-		(at 194.31 59.69 0)
+		(at 189.23 59.69 0)
 		(effects
 			(font
@@
 	)
 	(label "LCD_BACK"
-		(at 194.31 39.37 0)
+		(at 189.23 39.37 0)
 		(effects
 			(font
@@
 	)
 	(label "LCD_SCLK"
-		(at 194.31 49.53 0)
+		(at 189.23 49.53 0)
 		(effects
 			(font
@@
 	)
 	(label "HDI_SDA"
-		(at 236.22 41.91 0)
+		(at 214.63 39.37 0)
 		(effects
 			(font
@@
 	)
 	(label "LED_EN"
-		(at 236.22 46.99 0)
+		(at 214.63 44.45 0)
 		(effects
 			(font
@@
 	(hierarchical_label "{HID}"
 		(shape bidirectional)
-		(at 254 29.29 0)
+		(at 232.41 26.75 0)
 		(effects
 			(font
@@
 	(hierarchical_label "{LCD}"
 		(shape bidirectional)
-		(at 212.09 26.67 0)
-		(effects
-			(font
+		(at 207.01 26.67 0)
+		(effects
+			(font
