File: pcb/v2_mini_pcb/MCU.kicad_sch (KiCad schematic)
At the start: 20 parts, among them J5 TC2030, SW1 SW_Push, SW2 SW_Push

Commit message: vbus connection
Changed lines of the file:
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@@
+		)
+	)
+	(bus_entry
+		(at 88.9 52.07)
+		(size -2.54 2.54)
+		(stroke
+			(width 0)
+			(type default)
 		)
 	)
@@
 		)
 	)
+	(bus
+		(pts
+			(xy 88.9 46.99) (xy 88.9 52.07)
+		)
+		(stroke
+			(width 0)
+			(type default)
+		)
+	)
 	(wire
 		(pts
@@
 		(pts
 			(xy 229.87 44.45) (xy 214.63 44.45)
+		)
+		(stroke
+			(width 0)
+			(type default)
+		)
+	)
+	(wire
+		(pts
+			(xy 86.36 54.61) (xy 71.12 54.61)
 		)
 		(stroke
@@
 		)
 	)
+	(label "USB_VBUS_S"
+		(at 71.12 54.61 0)
+		(effects
+			(font
+				(size 1.27 1.27)
+			)
+			(justify left bottom)
+		)
+	)

Commit message: fix last erc errors
Connections:
- net LED_EN: now also U2.50 (GPIO39); no longer U2.14 (GPIO8)
Changed lines of the file:
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@@
-	)
-	(no_connect
-		(at 165.1 158.75)
 	)
 	(no_connect
@@
 	)
 	(no_connect
+		(at 78.74 133.35)
+	)
+	(no_connect
 		(at 137.16 175.26)
 	)
@@
 		)
 	)
-	(wire
-		(pts
-			(xy 62.23 133.35) (xy 78.74 133.35)
-		)
-		(stroke
-			(width 0)
-			(type default)
-		)
-	)
 	(bus
 		(pts
@@
 		(pts
 			(xy 172.72 100.33) (xy 184.15 100.33)
+		)
+		(stroke
+			(width 0)
+			(type default)
+		)
+	)
+	(wire
+		(pts
+			(xy 181.61 158.75) (xy 165.1 158.75)
 		)
 		(stroke
@@
 		)
 	)
+	(label "LED_EN"
+		(at 181.61 158.75 180)
+		(effects
+			(font
+				(size 1.27 1.27)
+			)
+			(justify right bottom)
+		)
+	)
 	(label "GNSS_TXD1"
 		(at 181.61 143.51 180)
@@
 		(effects
 			(font
-				(size 1.27 1.27)
-			)
-			(justify left bottom)
-		)
-	)
-	(label "LED_EN"
-		(at 62.23 133.35 0)
-		(effects
-			(font

Commit message: move jtag
Parts:
- added H4, H5, H6, H7: MountingHole_Pad, MountingHole:MountingHole_2.2mm_M2_Pad, symbol Mechanical:MountingHole_Pad
Connections:
- net GND: now also H4.1, H5.1, H6.1, H7.1

Commit message: fix drc problems nad d+d- and sd
Connections:
- net USB_DN: now also R17.2; no longer R10.2
- net USB_DP: now also R10.2; no longer R17.2
Changed lines of the file:
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@@
+		)
+	)
+	(label "USB_DN"
+		(at 124.46 191.77 90)
+		(effects
+			(font
+				(size 1.27 1.27)
+			)
+			(justify left bottom)
 		)
 	)
@@
 		)
 	)
+	(label "USB_DP"
+		(at 121.92 191.77 90)
+		(effects
+			(font
+				(size 1.27 1.27)
+			)
+			(justify left bottom)
+		)
+	)
 	(label "LCD_RN"
 		(at 189.23 34.29 0)
@@
 		)
 	)
-	(label "USB_DN"
-		(at 121.92 191.77 90)
-		(effects
-			(font
-				(size 1.27 1.27)
-			)
-			(justify left bottom)
-		)
-	)
 	(label "MAIN_SDA"
 		(at 62.23 130.81 0)
@@
 		(effects
 			(font
-				(size 1.27 1.27)
-			)
-			(justify left bottom)
-		)
-	)
-	(label "USB_DP"
-		(at 124.46 191.77 90)
-		(effects
-			(font

Commit message: jtag no 5v
Connections:
- net +3V3: no longer J5.1
- no-connect marks 13 -> 14
Changed lines of the file:
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@@
 	)
 	(no_connect
+		(at 328.93 88.9)
+	)
+	(no_connect
 		(at 165.1 102.87)
 	)
@@
 					(unit 1)
 				)
-			)
-		)
-	)
-	(symbol
-		(lib_id "power:+3V3")
-		(at 328.93 88.9 270)
-		(unit 1)
-		(body_style 1)
-		(exclude_from_sim no)
-		(in_bom yes)
-		(on_board yes)
-		(in_pos_files yes)
-		(dnp no)
-		(fields_autoplaced yes)
-		(property "Reference" "#PWR075"
-			(at 325.12 88.9 0)
-			(hide yes)
-			(show_name no)
-			(do_not_autoplace no)
-			(effects
-				(font
-					(size 1.27 1.27)
-				)
-			)
-		)
-		(property "Value" "+3V3"
-			(at 332.74 88.8999 90)
-			(show_name no)
-			(do_not_autoplace no)
-			(effects
-				(font
-					(size 1.27 1.27)
-				)
-				(justify left)
-			)
-		)
-		(property "Footprint" ""
-			(at 328.93 88.9 0)
-			(hide yes)
-			(show_name no)
-			(do_not_autoplace no)
-			(effects
-				(font
-					(size 1.27 1.27)
-				)
-			)
-		)
-		(property "Datasheet" ""
-			(at 328.93 88.9 0)
-			(hide yes)
-			(show_name no)
-			(do_not_autoplace no)
-			(effects
-				(font
-					(size 1.27 1.27)
-				)
-			)
-		)
-		(property "Description" "Power symbol creates a global label with name \"+3V3\""
-			(at 328.93 88.9 0)
-			(hide yes)
-			(show_name no)
-			(do_not_autoplace no)
-			(effects
-				(font
-					(size 1.27 1.27)
-				)
-			)
-		)
-		(pin "1"
-		)
-		(instances
-			(project "v2_mini"
-				(path "/4318b369-034c-40ef-a05b-b7d2541c0647/d810a1dc-5c9a-4ac6-8c4b-d9616121b31e"
-					(reference "#PWR075")
-					(unit 1)
-				)

Commit message: add power off schematic
Connections:
- net PWR_KILL_N: now reaches U2.14 (GPIO8)
- net PWR_INT_N: now reaches U2.49 (GPIO38)
- no-connect marks 14 -> 12
Other:
- moved on the sheet: H4, H5, H6, H7
Changed lines of the file:
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@@
 	)
 	(junction
-		(at 254 199.39)
+		(at 284.48 218.44)
 		(diameter 0)
 		(color 0 0 0 0)
@@
 	)
 	(junction
-		(at 247.65 199.39)
+		(at 278.13 218.44)
 		(diameter 0)
 		(color 0 0 0 0)
@@
 	)
 	(junction
-		(at 261.62 199.39)
+		(at 292.1 218.44)
 		(diameter 0)
 		(color 0 0 0 0)
@@
 	)
 	(no_connect
-		(at 165.1 161.29)
-	)
-	(no_connect
 		(at 165.1 115.57)
 	)
@@
 	)
 	(no_connect
-		(at 78.74 133.35)
-	)
-	(no_connect
 		(at 137.16 175.26)
 	)
@@
 	)
 	(bus_entry
+		(at 55.88 62.23)
+		(size -2.54 2.54)
+		(stroke
+			(width 0)
+			(type default)
+		)
+	)
+	(bus_entry
 		(at 88.9 36.83)
 		(size -2.54 2.54)
@@
 	)
 	(bus_entry
+		(at 55.88 67.31)
+		(size -2.54 2.54)
+		(stroke
+			(width 0)
+			(type default)
+		)
+	)
+	(bus_entry
 		(at 119.38 46.99)
 		(size -2.54 2.54)
@@
 	(wire
 		(pts
+			(xy 62.23 133.35) (xy 78.74 133.35)
+		)
+		(stroke
+			(width 0)
+			(type default)
+		)
+	)
+	(wire
+		(pts
 			(xy 165.1 148.59) (xy 181.61 148.59)
 		)
@@
 		)
 	)
+	(bus
+		(pts
+			(xy 55.88 57.15) (xy 55.88 67.31)
+		)
+		(stroke
+			(width 0)
+			(type default)
+		)
+	)
 	(wire
 		(pts
@@
 	(wire
 		(pts
-			(xy 254 199.39) (xy 261.62 199.39)
+			(xy 284.48 218.44) (xy 292.1 218.44)
 		)
 		(stroke
@@
 	(wire
 		(pts
+			(xy 53.34 64.77) (xy 38.1 64.77)
+		)
+		(stroke
+			(width 0)
+			(type default)
+		)
+	)
+	(wire
+		(pts
 			(xy 62.23 95.25) (xy 63.5 95.25)
 		)
@@
 	(wire
 		(pts
-			(xy 261.62 199.39) (xy 270.51 199.39)
+			(xy 292.1 218.44) (xy 300.99 218.44)
 		)
 		(stroke
@@
 	(wire
 		(pts
-			(xy 247.65 199.39) (xy 254 199.39)
+			(xy 278.13 218.44) (xy 284.48 218.44)
 		)
 		(stroke
@@
 	(wire
 		(pts
+			(xy 53.34 69.85) (xy 38.1 69.85)
+		)
+		(stroke
+			(width 0)
+			(type default)
+		)
+	)
+	(wire
+		(pts
 			(xy 62.23 130.81) (xy 78.74 130.81)
 		)
@@
 	(wire
 		(pts
+			(xy 165.1 161.29) (xy 181.61 161.29)
+		)
+		(stroke
+			(width 0)
+			(type default)
+		)
+	)
+	(wire
+		(pts
 			(xy 111.76 191.77) (xy 111.76 175.26)
 		)
@@
 		)
 	)
+	(label "PWR_INT_N"
+		(at 38.1 64.77 0)
+		(effects
+			(font
+				(size 1.27 1.27)
+			)
+			(justify left bottom)
+		)
+	)
 	(label "SD_CLK"
 		(at 163.83 34.29 0)
@@
 		)
 	)
+	(label "PWR_INT_N"
+		(at 181.61 161.29 180)
+		(effects
+			(font
+				(size 1.27 1.27)
+			)
+			(justify right bottom)
+		)
+	)
 	(label "IMU_CS_N"
 		(at 132.08 49.53 0)
@@
 		)
 	)
+	(label "PWR_KILL_N"
+		(at 38.1 69.85 0)
+		(effects
+			(font
+				(size 1.27 1.27)
+			)
+			(justify left bottom)
+		)
+	)
 	(label "SD_D0"
 		(at 106.68 191.77 90)
@@
 		)
 	)
+	(label "PWR_KILL_N"
+		(at 62.23 133.35 0)
+		(effects
+			(font
+				(size 1.27 1.27)
+			)
+			(justify left bottom)
+		)
+	)
 	(label "LCD_DC"
 		(at 62.23 161.29 0)
@@
 	(symbol
 		(lib_id "Mechanical:MountingHole_Pad")
-		(at 270.51 201.93 180)
+		(at 300.99 220.98 180)
 		(unit 1)
 		(body_style 1)
@@
 		(fields_autoplaced yes)
 		(property "Reference" "H7"
-			(at 273.05 201.9299 0)
+			(at 303.53 220.9799 0)
 			(show_name no)
 			(do_not_autoplace no)
@@
 		)
 		(property "Value" "MountingHole_Pad"
-			(at 273.05 204.4699 0)
+			(at 303.53 223.5199 0)
 			(show_name no)
 			(do_not_autoplace no)
@@
 		)
 		(property "Footprint" "MountingHole:MountingHole_2.2mm_M2_Pad"
-			(at 270.51 201.93 0)
+			(at 300.99 220.98 0)
 			(hide yes)
 			(show_name no)
@@
 		)
 		(property "Datasheet" ""
-			(at 270.51 201.93 0)
+			(at 300.99 220.98 0)
 			(hide yes)
 			(show_name no)
@@
 		)
 		(property "Description" "Mounting Hole with connection"
-			(at 270.51 201.93 0)
+			(at 300.99 220.98 0)
 			(hide yes)
 			(show_name no)
@@
 	(symbol
 		(lib_id "Mechanical:MountingHole_Pad")
-		(at 261.62 201.93 180)
+		(at 292.1 220.98 180)
 		(unit 1)
 		(body_style 1)
@@
 		(fields_autoplaced yes)
 		(property "Reference" "H6"
-			(at 264.16 201.9299 0)
+			(at 294.64 220.9799 0)
 			(show_name no)
 			(do_not_autoplace no)
@@
 		)
 		(property "Value" "MountingHole_Pad"
-			(at 264.16 204.4699 0)
+			(at 294.64 223.5199 0)
 			(show_name no)
 			(do_not_autoplace no)
@@
 		)
 		(property "Footprint" "MountingHole:MountingHole_2.2mm_M2_Pad"
-			(at 261.62 201.93 0)
+			(at 292.1 220.98 0)
 			(hide yes)
 			(show_name no)
@@
 		)
 		(property "Datasheet" ""
-			(at 261.62 201.93 0)
+			(at 292.1 220.98 0)
 			(hide yes)
 			(show_name no)
@@
 		)
 		(property "Description" "Mounting Hole with connection"
-			(at 261.62 201.93 0)
+			(at 292.1 220.98 0)
 			(hide yes)
 			(show_name no)
@@
 	(symbol
 		(lib_id "Mechanical:MountingHole_Pad")
-		(at 254 201.93 180)
+		(at 284.48 220.98 180)
 		(unit 1)
 		(body_style 1)
@@
 		(fields_autoplaced yes)
 		(property "Reference" "H5"
-			(at 256.54 201.9299 0)
+			(at 287.02 220.9799 0)
 			(show_name no)
 			(do_not_autoplace no)
@@
 		)
 		(property "Value" "MountingHole_Pad"
-			(at 256.54 204.4699 0)
+			(at 287.02 223.5199 0)
 			(show_name no)
 			(do_not_autoplace no)
@@
 		)
 		(property "Footprint" "MountingHole:MountingHole_2.2mm_M2_Pad"
-			(at 254 201.93 0)
+			(at 284.48 220.98 0)
 			(hide yes)
 			(show_name no)
@@
 		)
 		(property "Datasheet" ""
-			(at 254 201.93 0)
+			(at 284.48 220.98 0)
 			(hide yes)
 			(show_name no)
@@
 		)
 		(property "Description" "Mounting Hole with connection"
-			(at 254 201.93 0)
+			(at 284.48 220.98 0)
 			(hide yes)
 			(show_name no)
@@
 	(symbol
 		(lib_id "power:GND")
-		(at 247.65 199.39 180)
+		(at 278.13 218.44 180)
 		(unit 1)
 		(body_style 1)
@@
 		(fields_autoplaced yes)
 		(property "Reference" "#PWR089"
-			(at 247.65 193.04 0)
+			(at 278.13 212.09 0)
 			(hide yes)
 			(show_name no)
@@
 		)
 		(property "Value" "GND"
-			(at 247.65 194.31 0)
+			(at 278.13 213.36 0)
 			(show_name no)
 			(do_not_autoplace no)
@@
 		)
 		(property "Footprint" ""
-			(at 247.65 199.39 0)
+			(at 278.13 218.44 0)
 			(hide yes)
 			(show_name no)
@@
 		)
 		(property "Datasheet" ""
-			(at 247.65 199.39 0)
+			(at 278.13 218.44 0)
 			(hide yes)
 			(show_name no)
@@
 		)
 		(property "Description" "Power symbol creates a global label with name \"GND\" , ground"
-			(at 247.65 199.39 0)
+			(at 278.13 218.44 0)
 			(hide yes)
 			(show_name no)
@@
 	(symbol
 		(lib_id "Mechanical:MountingHole_Pad")
-		(at 247.65 201.93 180)
+		(at 278.13 220.98 180)
 		(unit 1)
 		(body_style 1)
@@
 		(fields_autoplaced yes)
 		(property "Reference" "H4"
-			(at 250.19 201.9299 0)
+			(at 280.67 220.9799 0)
 			(show_name no)
 			(do_not_autoplace no)
@@
 		)
 		(property "Value" "MountingHole_Pad"
-			(at 250.19 204.4699 0)
+			(at 280.67 223.5199 0)
 			(show_name no)
 			(do_not_autoplace no)
@@
 		)
 		(property "Footprint" "MountingHole:MountingHole_2.2mm_M2_Pad"
-			(at 247.65 201.93 0)
+			(at 278.13 220.98 0)
 			(hide yes)
 			(show_name no)
@@
 		)
 		(property "Datasheet" ""
-			(at 247.65 201.93 0)
+			(at 278.13 220.98 0)
 			(hide yes)
 			(show_name no)
@@
 		)
 		(property "Description" "Mounting Hole with connection"
-			(at 247.65 201.93 0)
+			(at 278.13 220.98 0)
 			(hide yes)
 			(show_name no)

Commit message: update bom
Parts:
- C10: DigiKey_PN (none) -> 311-1903-1-ND; JLCPCB_PN C45783 -> (none); LCSC C45783 -> (none); MPN CL21A226MAQNNNE -> CC0805MKX5R8BB226; Manufacturer Samsung Electro-Mechanics -> YAGEO; Supplier JLCPCB Basic -> DigiKey
- R10, R17, R30, R31: DigiKey_PN (none) -> 311-22.0LRCT-ND; MPN 0402WGF220JTCE -> RC0402FR-0722RL; Manufacturer (none) -> YAGEO; Power (none) -> 0.063W; Supplier (none) -> DigiKey; Temperature_Coefficient (none) -> ±100ppm/°C; Tolerance (none) -> 1%; Voltage (none) -> 50V
- R16, R21: DigiKey_PN (none) -> 311-5.10KLRCT-ND; MPN 0402WGF5101TCE -> RC0402FR-075K1L; Manufacturer (none) -> YAGEO; Power (none) -> 0.063W; Supplier (none) -> DigiKey; Temperature_Coefficient (none) -> ±100ppm/°C; Tolerance (none) -> 1%; Voltage (none) -> 50V
- R8, R9: DigiKey_PN (none) -> 311-10.0KLRCT-ND; MPN 0402WGF1002TCE -> RC0402FR-0710KL; Manufacturer (none) -> YAGEO; Power (none) -> 0.063W; Supplier (none) -> DigiKey; Temperature_Coefficient (none) -> ±100ppm/°C; Tolerance (none) -> 1%; Voltage (none) -> 50V
