File: pcb/v2_mini_pcb/v2_mini.kicad_pcb (KiCad board)
At the start: 6 copper layers, 70.8 x 36 mm, 109 parts, among them J1 Conn_Coaxial, J2 GTFP08441BEU, J3 SFV24R-2STE1HLF, J5 TC2030, J6 USB4105-GF-A, Q1 NTNS3164NZT5G, SW1 SW_Push, SW2 SW_Push, SW3 SW_Push, SW4 SW_Push, SW5 SW_Push, SW6 SW_Push, U1 UM980, U10 TPS63802DLAR, U3 SCH16T-K01-1, U4 LP5813ADRRR, U5 TCA9536ADTMR, U6 TPD4EUSB30, U8 BQ25622ERYKR, U9 MAX17048G_T10

Commit message: imu power
Parts:
- moved FB1 1.99 mm to (98.8, 82.8)
- moved FB2 1.99 mm to (98.8, 80.8)
Routing:
- net +3V3_IMU: track 9.81 -> 56.0 mm
- net +3V3_GNSS: track 42.0 -> 41.0 mm
Changed lines of the file:
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@@
 	(footprint "Inductor_SMD:L_0805_2012Metric"
 		(layer "F.Cu")
-		(at 98.8 80.8)
+		(at 98.81 82.79)
 		(descr "Inductor SMD 0805 (2012 Metric), square (rectangular) end terminal, IPC-7351 nominal, (Body size source: IPC-SM-782 page 80, https://www.pcb-3d.com/wordpress/wp-content/uploads/ipc-sm-782a_amendment_1_and_2.pdf)")
 		(tags "inductor")
@@
 	(footprint "Inductor_SMD:L_0805_2012Metric"
 		(layer "F.Cu")
-		(at 98.81 82.79)
+		(at 98.8 80.8)
 		(descr "Inductor SMD 0805 (2012 Metric), square (rectangular) end terminal, IPC-7351 nominal, (Body size source: IPC-SM-782 page 80, https://www.pcb-3d.com/wordpress/wp-content/uploads/ipc-sm-782a_amendment_1_and_2.pdf)")
 		(tags "inductor")
@@
 	)
 	(via
-		(at 99.7 81.19)
-		(size 0.5)
-		(drill 0.3)
-		(layers "F.Cu" "B.Cu")
-		(net "+3V3_GNSS")
-	)
-	(via
-		(at 99.72 80.46)
+		(at 99.78 83.19)
 		(size 0.5)
 		(drill 0.3)
@@
 	)
 	(via
-		(at 100.2 80.79)
+		(at 100.24 82.83)
 		(size 0.5)
 		(drill 0.3)
@@
 	)
 	(via
+		(at 99.8 82.47)
+		(size 0.5)
+		(drill 0.3)
+		(layers "F.Cu" "B.Cu")
+		(net "+3V3_GNSS")
+	)
+	(via
 		(at 103.52 102.7)
 		(size 0.5)
@@
 	)
 	(segment
-		(start 100.2 80.79)
-		(end 102.27 82.86)
-		(width 1)
-		(layer "In2.Cu")
-		(net "+3V3_GNSS")
-	)
-	(segment
 		(start 103.186041 102.383959)
-		(end 103.502082 102.7)
+		(end 103.09 102.287918)
 		(width 1)
 		(layer "In2.Cu")
@@
 	)
 	(segment
-		(start 100.2 80.79)
-		(end 99.72 80.79)
+		(start 103.09 102.287918)
+		(end 103.09 82.86)
 		(width 1)
 		(layer "In2.Cu")
@@
 	)
 	(segment
-		(start 103.09 82.86)
-		(end 103.09 102.287918)
+		(start 103.186041 102.383959)
+		(end 103.502082 102.7)
 		(width 1)
 		(layer "In2.Cu")
@@
 	)
 	(segment
-		(start 102.27 82.86)
-		(end 103.09 82.86)
-		(width 1)
-		(layer "In2.Cu")
-		(net "+3V3_GNSS")
-	)
-	(segment
-		(start 103.09 102.287918)
-		(end 103.186041 102.383959)
+		(start 103.09 82.86)
+		(end 99.88 82.86)
 		(width 1)
 		(layer "In2.Cu")
@@
 	)
 	(via
-		(at 99.78 83.19)
+		(at 99.7 81.19)
 		(size 0.5)
 		(drill 0.3)
@@
 	)
 	(via
-		(at 100.24 82.83)
+		(at 99.72 80.46)
 		(size 0.5)
 		(drill 0.3)
@@
 	)
 	(via
-		(at 131.03 98.4125)
+		(at 100.2 80.79)
 		(size 0.5)
 		(drill 0.3)
@@
 	)
 	(via
-		(at 131.05 83.38)
+		(at 131.03 98.4125)
 		(size 0.5)
 		(drill 0.3)
@@
 	)
 	(via
-		(at 130.23 98.4125)
+		(at 131.05 83.38)
 		(size 0.5)
 		(drill 0.3)
@@
 	)
 	(via
-		(at 99.8 82.47)
+		(at 130.23 98.4125)
 		(size 0.5)
 		(drill 0.3)
@@
 	)
 	(segment
+		(start 131.03 86.0825)
+		(end 131.03 98.4125)
+		(width 0.4)
+		(layer "B.Cu")
+		(net "+3V3_IMU")
+	)
+	(segment
+		(start 126.02 84.35)
+		(end 128.14 84.35)
+		(width 0.4)
+		(layer "In2.Cu")
+		(net "+3V3_IMU")
+	)
+	(segment
+		(start 100.05 80.79)
+		(end 99.72 80.46)
+		(width 0.4)
+		(layer "In2.Cu")
+		(net "+3V3_IMU")
+	)
+	(segment
 		(start 128.66 83.83)
 		(end 128.14 84.35)
@@
 	)
 	(segment
+		(start 99.8 81.19)
+		(end 100.2 80.79)
+		(width 0.4)
+		(layer "In2.Cu")
+		(net "+3V3_IMU")
+	)
+	(segment
+		(start 125.12 80.27)
+		(end 125.12 83.63)
+		(width 0.4)
+		(layer "In2.Cu")
+		(net "+3V3_IMU")
+	)
+	(segment
+		(start 125.3 83.63)
+		(end 126.02 84.35)
+		(width 0.4)
+		(layer "In2.Cu")
+		(net "+3V3_IMU")
+	)
+	(segment
+		(start 125.12 83.63)
+		(end 125.3 83.63)
+		(width 0.4)
+		(layer "In2.Cu")
+		(net "+3V3_IMU")
+	)
+	(segment
 		(start 131.05 83.38)
 		(end 130.6 83.83)
@@
 	)
 	(segment
+		(start 100.2 80.79)
+		(end 100.05 80.79)
+		(width 0.4)
+		(layer "In2.Cu")
+		(net "+3V3_IMU")
+	)
+	(segment
 		(start 130.6 83.83)
 		(end 128.66 83.83)
@@
 		(layer "In2.Cu")
 		(net "+3V3_IMU")
+	)
+	(segment
+		(start 101.65 79.34)
+		(end 124.19 79.34)
+		(width 0.4)
+		(layer "In2.Cu")
+		(net "+3V3_IMU")
+	)
+	(segment
+		(start 100.2 80.79)
+		(end 101.65 79.34)
+		(width 0.4)
+		(layer "In2.Cu")
+		(net "+3V3_IMU")
+	)
+	(segment
+		(start 124.19 79.34)
+		(end 125.12 80.27)
+		(width 0.4)
+		(layer "In2.Cu")
+		(net "+3V3_IMU")
+	)
+	(segment
+		(start 99.7 81.19)
+		(end 99.8 81.19)
+		(width 0.4)
+		(layer "In2.Cu")
+		(net "+3V3_IMU")

Commit message: sd done
Parts:
- C13, C14, R19: moved to B.Cu
- moved J5 92.0 mm to (70.7, 113.3), turned to 90 degrees
- moved C13 63.8 mm to (122.9, 89.7), turned to -90 degrees
- moved R19 63.1 mm to (122.2, 88.2)
- moved C14 59.8 mm to (121.5, 90.9), turned to 90 degrees
- moved U5 54.5 mm to (122.7, 105.8)
- moved U4 26.7 mm to (130.9, 79.7)
- moved C28 17.9 mm to (120.9, 118.4)
Routing:
- net +3V3: track 46.0 -> 114.5 mm, vias 12 -> 15
- net /ESP32-S31 MCU/SD_D0: track 0.00 -> 46.1 mm, vias 0 -> 2
- net /ESP32-S31 MCU/SD_D1: track 0.00 -> 43.6 mm, vias 0 -> 2
- net /ESP32-S31 MCU/SD_CMD: track 0.00 -> 36.1 mm, vias 0 -> 2
- net /ESP32-S31 MCU/SD_D3: track 0.00 -> 35.0 mm, vias 0 -> 2
- net /ESP32-S31 MCU/SD_D2: track 0.00 -> 34.8 mm, vias 0 -> 2
- net /ESP32-S31 MCU/SD_CLK: track 0.00 -> 31.0 mm, vias 0 -> 2
- net Net-(J2-CLK): track 0.00 -> 6.18 mm, vias 0 -> 2
- net /ESP32-S31 MCU/IMU_RESET_N: track 59.5 -> 63.3 mm
- net /ESP32-S31 MCU/IMU_MISO: track 46.1 -> 45.4 mm
- net GND: vias 170 -> 178
