File: pcb/v2_mini_pcb/GNSS_Mini.kicad_sch (KiCad schematic)
At the start: 17 parts, among them J1 Conn_Coaxial, U1 UM980

Commit message: update bom
Parts:
- C35, C4, C5, C6, C7: DigiKey_PN (none) -> 445-14418-1-ND; JLCPCB_PN C15850 -> (none); LCSC C15850 -> (none); MPN CL21A106KAYNNNE -> C2012X5R1V106K125AC; Manufacturer Samsung Electro-Mechanics -> TDK; Supplier JLCPCB Basic -> DigiKey; Voltage 25V -> 35V
- R1, R2, R24: DigiKey_PN (none) -> 311-10.0KLRCT-ND; MPN 0402WGF1002TCE -> RC0402FR-0710KL; Manufacturer (none) -> YAGEO; Power (none) -> 0.063W; Supplier (none) -> DigiKey; Temperature_Coefficient (none) -> ±100ppm/°C; Tolerance (none) -> 1%; Voltage (none) -> 50V
