File: pcb/v2_mini_pcb/Storage_Display.kicad_sch (KiCad schematic)
At the start: 12 parts, among them J2 GTFP08441BEU, J3 SFV24R-2STE1HLF, Q1 NTNS3164NZT5G

Commit message: finish v2_mini schematic
Parts:
- added R19: 22, symbol Device:R_Small_US
Connections:
- net SD_CLK: now also R19.1; no longer J2.5 (CLK)
- new net: J2.5 (CLK), R19.2
Changed lines of the file:
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@@
 	(wire
 		(pts
-			(xy 36.83 81.28) (xy 62.23 81.28)
+			(xy 36.83 81.28) (xy 53.34 81.28)
 		)
 		(stroke
@@
 	(wire
 		(pts
+			(xy 58.42 81.28) (xy 62.23 81.28)
+		)
+		(stroke
+			(width 0)
+			(type default)
+		)
+	)
+	(wire
+		(pts
 			(xy 176.53 81.28) (xy 187.96 81.28)
 		)
@@
 		)
 	)
-	(label "SD_D2"
+	(label "SD_D3"
 		(at 55.88 50.8 0)
 		(effects
@@
 					(unit 1)
 				)
+			)
+		)
+	)
+	(symbol
+		(lib_id "Device:R_Small_US")
+		(at 55.88 81.28 90)
+		(unit 1)
+		(body_style 1)
+		(exclude_from_sim no)
+		(in_bom yes)
+		(on_board yes)
+		(in_pos_files yes)
+		(dnp no)
+		(property "Reference" "R19"
+			(at 59.725 80.264 90)
+			(show_name no)
+			(do_not_autoplace no)
+			(effects
+				(font
+					(size 1.27 1.27)
+				)
+				(justify left)
+			)
+		)
+		(property "Value" "22"
+			(at 54.645 80.264 90)
+			(show_name no)
+			(do_not_autoplace no)
+			(effects
+				(font
+					(size 1.27 1.27)
+				)
+				(justify left)
+			)
+		)
+		(property "Footprint" ""
+			(at 55.88 81.28 0)
+			(hide yes)
+			(show_name no)
+			(do_not_autoplace no)
+			(effects
+				(font
+					(size 1.27 1.27)
+				)
+			)
+		)
+		(property "Datasheet" ""
+			(at 55.88 81.28 0)
+			(hide yes)
+			(show_name no)
+			(do_not_autoplace no)
+			(effects
+				(font
+					(size 1.27 1.27)
+				)
+			)
+		)
+		(property "Description" "Resistor, small US symbol"
+			(at 55.88 81.28 0)
+			(hide yes)
+			(show_name no)
+			(do_not_autoplace no)
+			(effects
+				(font
+					(size 1.27 1.27)
+				)
+			)
+		)
+		(pin "1"
+		)
+		(pin "2"
+		)
+		(instances
+			(project "v2_mini"
+				(path "/4318b369-034c-40ef-a05b-b7d2541c0647/0a25b8a8-ad00-432b-a1e7-4a7291f71ca1"
+					(reference "R19")
+					(unit 1)
+				)

Commit message: fix minor edc rules
Changed lines of the file:
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@@
 		)
 	)
-	(hierarchical_label "{SD}"
+	(hierarchical_label "{LCD}"
 		(shape bidirectional)
 		(at 231.14 20.4 0)

Commit message: add mpn and footprints for some
Parts:
- C13, C15, C22: footprint (none) -> Capacitor_SMD:C_01005_0402Metric; MPN (none) -> CL05B104KB54PNC
- C14, C23: footprint (none) -> Capacitor_SMD:C_0201_0603Metric; MPN (none) -> CL10A106KP8NNNC
Changed lines of the file:
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@@
+			)
+		)
+		(property "MPN" ""
+			(at 173.99 80.01 90)
+			(hide yes)
+			(show_name no)
+			(do_not_autoplace no)
+			(effects
+				(font
+					(size 1.27 1.27)
+				)
 			)
 		)
@@
 			)
 		)
+		(property "MPN" ""
+			(at 173.99 77.47 90)
+			(hide yes)
+			(show_name no)
+			(do_not_autoplace no)
+			(effects
+				(font
+					(size 1.27 1.27)
+				)
+			)
+		)
 		(pin "2"
 		)
@@
 			)
 		)
-		(property "Footprint" ""
+		(property "Footprint" "Capacitor_SMD:C_01005_0402Metric"
 			(at 171.45 71.12 0)
 			(hide yes)
@@
 		)
 		(property "Description" "Unpolarized capacitor, small symbol"
+			(at 171.45 71.12 0)
+			(hide yes)
+			(show_name no)
+			(do_not_autoplace no)
+			(effects
+				(font
+					(size 1.27 1.27)
+				)
+			)
+		)
+		(property "MPN" "CL05B104KB54PNC"
 			(at 171.45 71.12 0)
 			(hide yes)
@@
 			)
 		)
+		(property "MPN" ""
+			(at 166.37 60.96 90)
+			(hide yes)
+			(show_name no)
+			(do_not_autoplace no)
+			(effects
+				(font
+					(size 1.27 1.27)
+				)
+			)
+		)
 		(pin "D"
 		)
@@
 			)
 		)
-		(property "Footprint" ""
+		(property "Footprint" "Capacitor_SMD:C_01005_0402Metric"
 			(at 99.06 73.66 0)
 			(hide yes)
@@
 		)
 		(property "Description" "Unpolarized capacitor, small symbol"
+			(at 99.06 73.66 0)
+			(hide yes)
+			(show_name no)
+			(do_not_autoplace no)
+			(effects
+				(font
+					(size 1.27 1.27)
+				)
+			)
+		)
+		(property "MPN" "CL05B104KB54PNC"
 			(at 99.06 73.66 0)
 			(hide yes)
@@
 			)
 		)
+		(property "MPN" ""
+			(at 80.01 88.9 0)
+			(hide yes)
+			(show_name no)
+			(do_not_autoplace no)
+			(effects
+				(font
+					(size 1.27 1.27)
+				)
+			)
+		)
 		(pin "1"
 		)
@@
 			)
 		)
+		(property "MPN" ""
+			(at 198.12 96.52 0)
+			(hide yes)
+			(show_name no)
+			(do_not_autoplace no)
+			(effects
+				(font
+					(size 1.27 1.27)
+				)
+			)
+		)
 		(pin "20"
 		)
@@
 			)
 		)
+		(property "MPN" ""
+			(at 165.1 53.34 0)
+			(hide yes)
+			(show_name no)
+			(do_not_autoplace no)
+			(effects
+				(font
+					(size 1.27 1.27)
+				)
+			)
+		)
 		(pin "2"
 		)
@@
 			)
 		)
-		(property "Footprint" ""
+		(property "Footprint" "Capacitor_SMD:C_0201_0603Metric"
 			(at 177.8 71.12 0)
 			(hide yes)
@@
 		)
 		(property "Description" "Unpolarized capacitor, small symbol"
+			(at 177.8 71.12 0)
+			(hide yes)
+			(show_name no)
+			(do_not_autoplace no)
+			(effects
+				(font
+					(size 1.27 1.27)
+				)
+			)
+		)
+		(property "MPN" "CL10A106KP8NNNC"
 			(at 177.8 71.12 0)
 			(hide yes)
@@
 			)
 		)
-		(property "Footprint" ""
+		(property "Footprint" "Capacitor_SMD:C_0201_0603Metric"
 			(at 109.22 73.66 0)
 			(hide yes)
@@
 			)
 		)
+		(property "MPN" "CL10A106KP8NNNC"
+			(at 109.22 73.66 0)
+			(hide yes)
+			(show_name no)
+			(do_not_autoplace no)
+			(effects
+				(font
+					(size 1.27 1.27)
+				)
+			)
+		)
 		(pin "1"
 		)
@@
 			)
 		)
-		(property "Footprint" ""
+		(property "Footprint" "Capacitor_SMD:C_01005_0402Metric"
 			(at 163.83 71.12 0)
 			(hide yes)
@@
 			)
 		)
+		(property "MPN" "CL05B104KB54PNC"
+			(at 163.83 71.12 0)
+			(hide yes)
+			(show_name no)
+			(do_not_autoplace no)
+			(effects
+				(font
+					(size 1.27 1.27)
+				)
+			)
+		)
 		(pin "1"
 		)
@@
 			)
 		)
+		(property "MPN" ""
+			(at 173.99 63.5 90)
+			(hide yes)
+			(show_name no)
+			(do_not_autoplace no)
+			(effects
+				(font
+					(size 1.27 1.27)
+				)
+			)
+		)
 		(pin "2"
 		)
@@
 			(hide yes)
 			(show_name no)
+			(do_not_autoplace no)
+			(effects
+				(font
+					(size 1.27 1.27)
+				)
+			)
+		)
+		(property "MPN" ""
+			(at 55.88 81.28 90)
+			(hide yes)
+			(show_name no)

Commit message: finish off mpn and footprints
Parts:
- C13, C15, C22: footprint Capacitor_SMD:C_01005_0402Metric -> Capacitor_SMD:C_0402_1005Metric; MPN CL05B104KB54PNC -> GRM155R71C104KA88D
- C14, C23: footprint Capacitor_SMD:C_0201_0603Metric -> Capacitor_SMD:C_0603_1608Metric; MPN CL10A106KP8NNNC -> GRM188R61A106ME69D
- J2: footprint GTFP08441BEU:AMPHENOL_GTFP08441BEU -> all:AMPHENOL_GTFP08441BEU; MPN (none) -> GTFP08441BEU
- J3: footprint SFV24R-2STE1HLF:AMPHENOL_SFV24R-2STE1HLF -> all:AMPHENOL_SFV24R-2STE1HLF; MPN (none) -> SFV24R-2STE1HLF
- Q1: footprint (none) -> Package_TO_SOT_SMD:SOT-883; MPN (none) -> NTNS3164NZT5G
- R19: footprint (none) -> Resistor_SMD:R_0402_1005Metric; MPN (none) -> 0402WGF220JTCE
- R4: footprint (none) -> Resistor_SMD:R_0402_1005Metric; MPN (none) -> RC0402FR-0715RL
- R5: footprint (none) -> Resistor_SMD:R_0402_1005Metric; MPN (none) -> 0402WGF1003TCE
- R6, R7: footprint (none) -> Resistor_SMD:R_0402_1005Metric; MPN (none) -> 0402WGF1002TCE
Changed lines of the file:
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@@
 			)
 		)
-		(property "Footprint" ""
+		(property "Footprint" "Resistor_SMD:R_0402_1005Metric"
 			(at 173.99 80.01 0)
 			(hide yes)
@@
 			)
 		)
-		(property "MPN" ""
+		(property "MPN" "0402WGF1002TCE"
 			(at 173.99 80.01 90)
 			(hide yes)
@@
 			)
 		)
-		(property "Footprint" ""
+		(property "Footprint" "Resistor_SMD:R_0402_1005Metric"
 			(at 173.99 77.47 0)
 			(hide yes)
@@
 			)
 		)
-		(property "MPN" ""
+		(property "MPN" "0402WGF1002TCE"
 			(at 173.99 77.47 90)
 			(hide yes)
@@
 			)
 		)
-		(property "Footprint" "Capacitor_SMD:C_01005_0402Metric"
+		(property "Footprint" "Capacitor_SMD:C_0402_1005Metric"
 			(at 171.45 71.12 0)
 			(hide yes)
@@
 			)
 		)
-		(property "MPN" "CL05B104KB54PNC"
+		(property "MPN" "GRM155R71C104KA88D"
 			(at 171.45 71.12 0)
 			(hide yes)
@@
 			)
 		)
-		(property "Footprint" ""
+		(property "Footprint" "Package_TO_SOT_SMD:SOT-883"
 			(at 168.91 66.04 0)
 			(hide yes)
@@
 			)
 		)
-		(property "MPN" ""
+		(property "MPN" "NTNS3164NZT5G"
 			(at 166.37 60.96 90)
 			(hide yes)
@@
 			)
 		)
-		(property "Footprint" "Capacitor_SMD:C_01005_0402Metric"
+		(property "Footprint" "Capacitor_SMD:C_0402_1005Metric"
 			(at 99.06 73.66 0)
 			(hide yes)
@@
 			)
 		)
-		(property "MPN" "CL05B104KB54PNC"
+		(property "MPN" "GRM155R71C104KA88D"
 			(at 99.06 73.66 0)
 			(hide yes)
@@
 			)
 		)
-		(property "Footprint" "GTFP08441BEU:AMPHENOL_GTFP08441BEU"
+		(property "Footprint" "all:AMPHENOL_GTFP08441BEU"
 			(at 80.01 88.9 0)
 			(hide yes)
@@
 			)
 		)
-		(property "MPN" ""
+		(property "MPN" "GTFP08441BEU"
 			(at 80.01 88.9 0)
 			(hide yes)
@@
 			)
 		)
-		(property "Footprint" "SFV24R-2STE1HLF:AMPHENOL_SFV24R-2STE1HLF"
+		(property "Footprint" "all:AMPHENOL_SFV24R-2STE1HLF"
 			(at 198.12 96.52 0)
 			(hide yes)
@@
 			)
 		)
-		(property "MPN" ""
+		(property "MPN" "SFV24R-2STE1HLF"
 			(at 198.12 96.52 0)
 			(hide yes)
@@
 			)
 		)
-		(property "Footprint" ""
+		(property "Footprint" "Resistor_SMD:R_0402_1005Metric"
 			(at 165.1 53.34 0)
 			(hide yes)
@@
 			)
 		)
-		(property "MPN" ""
+		(property "MPN" "0402WGF1003TCE"
 			(at 165.1 53.34 0)
 			(hide yes)
@@
 			)
 		)
-		(property "Footprint" "Capacitor_SMD:C_0201_0603Metric"
+		(property "Footprint" "Capacitor_SMD:C_0603_1608Metric"
 			(at 177.8 71.12 0)
 			(hide yes)
@@
 			)
 		)
-		(property "MPN" "CL10A106KP8NNNC"
+		(property "MPN" "GRM188R61A106ME69D"
 			(at 177.8 71.12 0)
 			(hide yes)
@@
 			)
 		)
-		(property "Footprint" "Capacitor_SMD:C_0201_0603Metric"
+		(property "Footprint" "Capacitor_SMD:C_0603_1608Metric"
 			(at 109.22 73.66 0)
 			(hide yes)
@@
 			)
 		)
-		(property "MPN" "CL10A106KP8NNNC"
+		(property "MPN" "GRM188R61A106ME69D"
 			(at 109.22 73.66 0)
 			(hide yes)
@@
 			)
 		)
-		(property "Footprint" "Capacitor_SMD:C_01005_0402Metric"
+		(property "Footprint" "Capacitor_SMD:C_0402_1005Metric"
 			(at 163.83 71.12 0)
 			(hide yes)
@@
 			)
 		)
-		(property "MPN" "CL05B104KB54PNC"
+		(property "MPN" "GRM155R71C104KA88D"
 			(at 163.83 71.12 0)
 			(hide yes)
@@
 			)
 		)
-		(property "Footprint" ""
+		(property "Footprint" "Resistor_SMD:R_0402_1005Metric"
 			(at 173.99 63.5 0)
 			(hide yes)
@@
 			)
 		)
-		(property "MPN" ""
+		(property "MPN" "RC0402FR-0715RL"
 			(at 173.99 63.5 90)
 			(hide yes)
@@
 			)
 		)
-		(property "Footprint" ""
+		(property "Footprint" "Resistor_SMD:R_0402_1005Metric"
 			(at 55.88 81.28 0)
 			(hide yes)
@@
 			)
 		)
-		(property "MPN" ""
+		(property "MPN" "0402WGF220JTCE"
 			(at 55.88 81.28 90)
 			(hide yes)

Commit message: finish footprint matching
Parts:
- C13, C15, C22: Dielectric (none) -> X7R; JLCPCB_PN (none) -> C1525; LCSC (none) -> C1525; MPN GRM155R71C104KA88D -> CL05B104KO5NNNC; Manufacturer (none) -> Samsung Electro-Mechanics; Supplier (none) -> JLCPCB Basic; Tolerance (none) -> 10%; Voltage (none) -> 16V
- C14, C23: Dielectric (none) -> X5R; JLCPCB_PN (none) -> C19702; LCSC (none) -> C19702; MPN GRM188R61A106ME69D -> CL10A106KP8NNNC; Manufacturer (none) -> Samsung Electro-Mechanics; Supplier (none) -> JLCPCB Basic; Tolerance (none) -> 10%; Voltage (none) -> 10V
- J2, J3: MANUFACTURER Amphenol -> (none); Manufacturer (none) -> Amphenol

Commit message: done with lcd pcb
Connections:
- net GND: now also Q1.2 (S); no longer Q1.S
- net LCD_BACK: now also Q1.1 (G); no longer Q1.G
- net at R4.1: now also Q1.3 (D); no longer Q1.D
Changed lines of the file:
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@@
 			)
 		)
-		(pin "D"
+		(pin "1"
 		)
-		(pin "G"
+		(pin "2"
 		)
-		(pin "S"
+		(pin "3"
 		)
 		(instances

Commit message: update bom
Parts:
- C14, C23: DigiKey_PN (none) -> 1276-CL10A106KP8NNNDCT-ND; JLCPCB_PN C19702 -> (none); LCSC C19702 -> (none); MPN CL10A106KP8NNNC -> CL10A106KP8NNND; Supplier JLCPCB Basic -> DigiKey
- R19: DigiKey_PN (none) -> 311-22.0LRCT-ND; MPN 0402WGF220JTCE -> RC0402FR-0722RL; Manufacturer (none) -> YAGEO; Power (none) -> 0.063W; Supplier (none) -> DigiKey; Temperature_Coefficient (none) -> ±100ppm/°C; Tolerance (none) -> 1%; Voltage (none) -> 50V
- R5: DigiKey_PN (none) -> 311-100KLRCT-ND; MPN 0402WGF1003TCE -> RC0402FR-07100KL; Manufacturer (none) -> YAGEO; Power (none) -> 0.063W; Supplier (none) -> DigiKey; Temperature_Coefficient (none) -> ±100ppm/°C; Tolerance (none) -> 1%; Voltage (none) -> 50V
- R6, R7: DigiKey_PN (none) -> 311-10.0KLRCT-ND; MPN 0402WGF1002TCE -> RC0402FR-0710KL; Manufacturer (none) -> YAGEO; Power (none) -> 0.063W; Supplier (none) -> DigiKey; Temperature_Coefficient (none) -> ±100ppm/°C; Tolerance (none) -> 1%; Voltage (none) -> 50V
Changed lines of the file:
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@@
 			)
 		)
-		(property "Datasheet" ""
+		(property "Datasheet" "https://www.yageogroup.com/component-documentation/download/specsheet/RC0402FR-0710KL"
 			(at 173.99 80.01 0)
 			(hide yes)
@@
 			)
 		)
-		(property "MPN" "0402WGF1002TCE"
+		(property "MPN" "RC0402FR-0710KL"
 			(at 173.99 80.01 90)
 			(hide yes)
@@
 			)
 		)
+    (property "Manufacturer" "YAGEO" (at 173.99 80.01 0)
+      (effects (font (size 1.27 1.27)) (hide yes))
+    )
+    (property "DigiKey_PN" "311-10.0KLRCT-ND" (at 173.99 80.01 0)
+      (effects (font (size 1.27 1.27)) (hide yes))
+    )
+    (property "Supplier" "DigiKey" (at 173.99 80.01 0)
+      (effects (font (size 1.27 1.27)) (hide yes))
+    )
+    (property "Voltage" "50V" (at 173.99 80.01 0)
+      (effects (font (size 1.27 1.27)) (hide yes))
+    )
+    (property "Tolerance" "1%" (at 173.99 80.01 0)
+      (effects (font (size 1.27 1.27)) (hide yes))
+    )
+    (property "Power" "0.063W" (at 173.99 80.01 0)
+      (effects (font (size 1.27 1.27)) (hide yes))
+    )
+    (property "Temperature_Coefficient" "±100ppm/°C" (at 173.99 80.01 0)
+      (effects (font (size 1.27 1.27)) (hide yes))
+    )
 		(pin "2"
 		)
@@
 			)
 		)
-		(property "Datasheet" ""
+		(property "Datasheet" "https://www.yageogroup.com/component-documentation/download/specsheet/RC0402FR-0710KL"
 			(at 173.99 77.47 0)
 			(hide yes)
@@
 			)
 		)
-		(property "MPN" "0402WGF1002TCE"
+		(property "MPN" "RC0402FR-0710KL"
 			(at 173.99 77.47 90)
 			(hide yes)
@@
 			)
 		)
+    (property "Manufacturer" "YAGEO" (at 173.99 77.47 0)
+      (effects (font (size 1.27 1.27)) (hide yes))
+    )
+    (property "DigiKey_PN" "311-10.0KLRCT-ND" (at 173.99 77.47 0)
+      (effects (font (size 1.27 1.27)) (hide yes))
+    )
+    (property "Supplier" "DigiKey" (at 173.99 77.47 0)
+      (effects (font (size 1.27 1.27)) (hide yes))
+    )
+    (property "Voltage" "50V" (at 173.99 77.47 0)
+      (effects (font (size 1.27 1.27)) (hide yes))
+    )
+    (property "Tolerance" "1%" (at 173.99 77.47 0)
+      (effects (font (size 1.27 1.27)) (hide yes))
+    )
+    (property "Power" "0.063W" (at 173.99 77.47 0)
+      (effects (font (size 1.27 1.27)) (hide yes))
+    )
+    (property "Temperature_Coefficient" "±100ppm/°C" (at 173.99 77.47 0)
+      (effects (font (size 1.27 1.27)) (hide yes))
+    )
 		(pin "2"
 		)
@@
 			)
 		)
-		(property "Datasheet" ""
+		(property "Datasheet" "https://www.yageogroup.com/component-documentation/download/specsheet/RC0402FR-07100KL"
 			(at 165.1 53.34 0)
 			(hide yes)
@@
 			)
 		)
-		(property "MPN" "0402WGF1003TCE"
+		(property "MPN" "RC0402FR-07100KL"
 			(at 165.1 53.34 0)
 			(hide yes)
@@
 			)
 		)
+    (property "Manufacturer" "YAGEO" (at 165.1 53.34 0)
+      (effects (font (size 1.27 1.27)) (hide yes))
+    )
+    (property "DigiKey_PN" "311-100KLRCT-ND" (at 165.1 53.34 0)
+      (effects (font (size 1.27 1.27)) (hide yes))
+    )
+    (property "Supplier" "DigiKey" (at 165.1 53.34 0)
+      (effects (font (size 1.27 1.27)) (hide yes))
+    )
+    (property "Voltage" "50V" (at 165.1 53.34 0)
+      (effects (font (size 1.27 1.27)) (hide yes))
+    )
+    (property "Tolerance" "1%" (at 165.1 53.34 0)
+      (effects (font (size 1.27 1.27)) (hide yes))
+    )
+    (property "Power" "0.063W" (at 165.1 53.34 0)
+      (effects (font (size 1.27 1.27)) (hide yes))
+    )
+    (property "Temperature_Coefficient" "±100ppm/°C" (at 165.1 53.34 0)
+      (effects (font (size 1.27 1.27)) (hide yes))
+    )
 		(pin "2"
 		)
@@
 			)
 		)
-		(property "Datasheet" ""
+		(property "Datasheet" "https://product.samsungsem.com/mlcc/CL10A106KP8NNN.do"
 			(at 177.8 71.12 0)
 			(hide yes)
@@
 			)
 		)
-		(property "MPN" "CL10A106KP8NNNC"
+		(property "MPN" "CL10A106KP8NNND"
 			(at 177.8 71.12 0)
 			(hide yes)
@@
 			)
 		)
-		(property "LCSC" "C19702"
-			(at 177.8 71.12 0)
-			(hide yes)
-			(show_name no)
-			(do_not_autoplace no)
-			(effects
-				(font
-					(size 1.27 1.27)
-				)
-			)
-		)
-		(property "JLCPCB_PN" "C19702"
-			(at 177.8 71.12 0)
-			(hide yes)
-			(show_name no)
-			(do_not_autoplace no)
-			(effects
-				(font
-					(size 1.27 1.27)
-				)
-			)
-		)
-		(property "Supplier" "JLCPCB Basic"
+		(property "Supplier" "DigiKey"
 			(at 177.8 71.12 0)
 			(hide yes)
@@
 			)
 		)
+    (property "DigiKey_PN" "1276-CL10A106KP8NNNDCT-ND" (at 177.8 71.12 0)
+      (effects (font (size 1.27 1.27)) (hide yes))
+    )
 		(pin "1"
 		)
@@
 			)
 		)
-		(property "Datasheet" ""
+		(property "Datasheet" "https://product.samsungsem.com/mlcc/CL10A106KP8NNN.do"
 			(at 109.22 73.66 0)
 			(hide yes)
@@
 			)
 		)
-		(property "MPN" "CL10A106KP8NNNC"
+		(property "MPN" "CL10A106KP8NNND"
 			(at 109.22 73.66 0)
 			(hide yes)
@@
 			)
 		)
-		(property "LCSC" "C19702"
-			(at 109.22 73.66 0)
-			(hide yes)
-			(show_name no)
-			(do_not_autoplace no)
-			(effects
-				(font
-					(size 1.27 1.27)
-				)
-			)
-		)
-		(property "JLCPCB_PN" "C19702"
-			(at 109.22 73.66 0)
-			(hide yes)
-			(show_name no)
-			(do_not_autoplace no)
-			(effects
-				(font
-					(size 1.27 1.27)
-				)
-			)
-		)
-		(property "Supplier" "JLCPCB Basic"
+		(property "Supplier" "DigiKey"
 			(at 109.22 73.66 0)
 			(hide yes)
@@
 			)
 		)
+    (property "DigiKey_PN" "1276-CL10A106KP8NNNDCT-ND" (at 109.22 73.66 0)
+      (effects (font (size 1.27 1.27)) (hide yes))
+    )
 		(pin "1"
 		)
@@
 			)
 		)
-		(property "Datasheet" ""
+		(property "Datasheet" "https://www.yageogroup.com/component-documentation/download/specsheet/RC0402FR-0722RL"
 			(at 55.88 81.28 0)
 			(hide yes)
@@
 			)
 		)
-		(property "MPN" "0402WGF220JTCE"
+		(property "MPN" "RC0402FR-0722RL"
 			(at 55.88 81.28 90)
 			(hide yes)
@@
 			)
 		)
+    (property "Manufacturer" "YAGEO" (at 55.88 81.28 0)
+      (effects (font (size 1.27 1.27)) (hide yes))
+    )
+    (property "DigiKey_PN" "311-22.0LRCT-ND" (at 55.88 81.28 0)
+      (effects (font (size 1.27 1.27)) (hide yes))
+    )
+    (property "Supplier" "DigiKey" (at 55.88 81.28 0)
+      (effects (font (size 1.27 1.27)) (hide yes))
+    )
+    (property "Voltage" "50V" (at 55.88 81.28 0)
+      (effects (font (size 1.27 1.27)) (hide yes))
+    )
+    (property "Tolerance" "1%" (at 55.88 81.28 0)
+      (effects (font (size 1.27 1.27)) (hide yes))
+    )
+    (property "Power" "0.063W" (at 55.88 81.28 0)
+      (effects (font (size 1.27 1.27)) (hide yes))
+    )
+    (property "Temperature_Coefficient" "±100ppm/°C" (at 55.88 81.28 0)
+      (effects (font (size 1.27 1.27)) (hide yes))
+    )
 		(pin "1"
 		)
